Commit message: updated crab model with Adam's latest 3D printed model and simplified collision geometry

File: crab.urdf (robot description, URDF)
Before this commit: robot crab_robot, 73 links, 72 joints
Links:
- removed link back__sensor_link
- removed link back_left__base_link
- removed link back_left__cluster_1_base_link
- removed link back_left__cluster_1_distal_link
- removed link back_left__cluster_1_end_link
- removed link back_left__cluster_1_proximal_link
- removed link back_left__cluster_2_base_link
- removed link back_left__cluster_2_distal_link
- removed link back_left__cluster_2_end_link
- removed link back_left__cluster_2_proximal_link
- removed link back_left__cluster_3_base_link
- removed link back_left__cluster_3_distal_link
- removed link back_left__cluster_3_end_link
- removed link back_left__cluster_3_mid_link
- removed link back_left__cluster_3_proximal_link
- removed link back_left__cluster_3_wrist_link
- removed link back_left__foot_link
- removed link back_right__base_link
- removed link back_right__cluster_1_base_link
- removed link back_right__cluster_1_distal_link
- removed link back_right__cluster_1_end_link
- removed link back_right__cluster_1_proximal_link
- removed link back_right__cluster_2_base_link
- removed link back_right__cluster_2_distal_link
- removed link back_right__cluster_2_end_link
- removed link back_right__cluster_2_proximal_link
- removed link back_right__cluster_3_base_link
- removed link back_right__cluster_3_distal_link
- removed link back_right__cluster_3_end_link
- removed link back_right__cluster_3_mid_link
- removed link back_right__cluster_3_proximal_link
- removed link back_right__cluster_3_wrist_link
- removed link back_right__foot_link
- removed link base_footprint
- removed link bottom_lidar_link
- removed link front_left__base_link
- removed link front_left__cluster_1_base_link
- removed link front_left__cluster_1_distal_link
- removed link front_left__cluster_1_end_link
- removed link front_left__cluster_1_proximal_link
- removed link front_left__cluster_2_base_link
- removed link front_left__cluster_2_distal_link
- removed link front_left__cluster_2_end_link
- removed link front_left__cluster_2_proximal_link
- removed link front_left__cluster_3_base_link
- removed link front_left__cluster_3_distal_link
- removed link front_left__cluster_3_end_link
- removed link front_left__cluster_3_mid_link
- removed link front_left__cluster_3_proximal_link
- removed link front_left__cluster_3_wrist_link
- removed link front_left__foot_link
- removed link front_left__sensor_link
- removed link front_right__base_link
- removed link front_right__cluster_1_base_link
- removed link front_right__cluster_1_distal_link
- removed link front_right__cluster_1_end_link
- removed link front_right__cluster_1_proximal_link
- removed link front_right__cluster_2_base_link
- removed link front_right__cluster_2_distal_link
- removed link front_right__cluster_2_end_link
- removed link front_right__cluster_2_proximal_link
- removed link front_right__cluster_3_base_link
- removed link front_right__cluster_3_distal_link
- removed link front_right__cluster_3_end_link
- removed link front_right__cluster_3_mid_link
- removed link front_right__cluster_3_proximal_link
- removed link front_right__cluster_3_wrist_link
- removed link front_right__foot_link
- removed link front_right__sensor_link
- removed link left__sensor_link
- removed link right__sensor_link
- removed link top_lidar_link
- added link arm1_foot_link, mass 1e-10; collision box size=0.15 0.15 0.04; visual box size=0.15 0.15 0.04
- added link arm1_link1, mass 0.935223157536645; visual mesh filename=arm1_link1.STL
- added link arm1_link2, mass 0.792615281561028; collision cylinder length=0.05 radius=0.04; visual mesh filename=arm1_link2.STL
- added link arm1_link3, mass 0.914578646343626; collision cylinder length=0.05 radius=0.03; visual mesh filename=arm1_link3.STL
- added link arm1_link4, mass 0.441334804948817; collision cylinder length=0.05 radius=0.03; visual mesh filename=arm1_link4.STL
- added link arm1_link5, mass 0.632159217766391; collision cylinder length=0.07 radius=0.025; visual mesh filename=arm1_link5.STL
- added link arm1_link6, mass 0.174644981988622; collision cylinder length=0.05 radius=0.02; visual mesh filename=arm1_link6.STL
- added link arm1_link7, mass 0.0367655989629361; visual mesh filename=arm1_link7.STL
- added link arm2_foot_link, mass 1e-10; collision box size=0.15 0.15 0.04; visual box size=0.15 0.15 0.04
- added link arm2_link1, mass 0.935223157536645; visual mesh filename=arm2_link1.STL
- added link arm2_link2, mass 0.792615281561028; collision cylinder length=0.05 radius=0.04; visual mesh filename=arm2_link2.STL
- added link arm2_link3, mass 0.914578646343627; collision cylinder length=0.05 radius=0.03; visual mesh filename=arm2_link3.STL
- added link arm2_link4, mass 0.441334804948817; collision cylinder length=0.05 radius=0.03; visual mesh filename=arm2_link4.STL
- added link arm2_link5, mass 0.632159217766392; collision cylinder length=0.07 radius=0.025; visual mesh filename=arm2_link5.STL
- added link arm2_link6, mass 0.174644982031482; collision cylinder length=0.05 radius=0.02; visual mesh filename=arm2_link6.STL
- added link arm2_link7, mass 0.0367655989629361; visual mesh filename=arm2_link7.STL
- added link arm3_foot_link, mass 1e-10; collision box size=0.15 0.15 0.04; visual box size=0.15 0.15 0.04
- added link arm3_link1, mass 0.935223157536645; visual mesh filename=arm3_link1.STL
- added link arm3_link2, mass 0.792615281561028; collision cylinder length=0.05 radius=0.04; visual mesh filename=arm3_link2.STL
- added link arm3_link3, mass 0.914578646343627; collision cylinder length=0.05 radius=0.03; visual mesh filename=arm3_link3.STL
- added link arm3_link4, mass 0.441334804948817; collision cylinder length=0.05 radius=0.03; visual mesh filename=arm3_link4.STL
- added link arm3_link5, mass 0.632159217766391; collision cylinder length=0.07 radius=0.025; visual mesh filename=arm3_link5.STL
- added link arm3_link6, mass 0.174644981988622; collision cylinder length=0.05 radius=0.02; visual mesh filename=arm3_link6.STL
- added link arm3_link7, mass 0.0367655989629361; visual mesh filename=arm3_link7.STL
- added link arm4_foot_link, mass 1e-10; collision box size=0.15 0.15 0.04; visual box size=0.15 0.15 0.04
- added link arm4_link1, mass 0.935223157536645; visual mesh filename=arm4_link1.STL
- added link arm4_link2, mass 0.792615281561028; collision cylinder length=0.05 radius=0.04; visual mesh filename=arm4_link2.STL
- added link arm4_link3, mass 0.914578646343627; collision cylinder length=0.05 radius=0.03; visual mesh filename=arm4_link3.STL
- added link arm4_link4, mass 0.441334804948817; collision cylinder length=0.05 radius=0.03; visual mesh filename=arm4_link4.STL
- added link arm4_link5, mass 0.63215921776639; collision cylinder length=0.07 radius=0.025; visual mesh filename=arm4_link5.STL
- added link arm4_link6, mass 0.174644981988622; collision cylinder length=0.05 radius=0.02; visual mesh filename=arm4_link6.STL
- added link arm4_link7, mass 0.0367655989629361; visual mesh filename=arm4_link7.STL
- added link back_sensor_link, mass 1e-10; visual box size=0.01 0.06 0.04
- added link front_sensor_link, mass 1e-10; visual box size=0.01 0.06 0.04
- link base_link: mass 100 -> 11.6672712209699; geometry collision box size=0.4 0.4 0.15; visual mesh filename=base_link.STL
Joints:
- removed joint back_left__cluster_1_base_fix
- removed joint back_left__cluster_1_end_joint
- removed joint back_left__cluster_1_pitch
- removed joint back_left__cluster_1_roll
- removed joint back_left__cluster_2_base_fix
- removed joint back_left__cluster_2_end_joint
- removed joint back_left__cluster_2_pitch
- removed joint back_left__cluster_2_roll
- removed joint back_left__cluster_3_base_fix
- removed joint back_left__cluster_3_end_joint
- removed joint back_left__cluster_3_mid_joint
- removed joint back_left__cluster_3_pitch
- removed joint back_left__cluster_3_roll
- removed joint back_left__cluster_3_wrist
- removed joint back_left__cluster_3_wrist_link_foot_joint
- removed joint back_right__cluster_1_base_fix
- removed joint back_right__cluster_1_end_joint
- removed joint back_right__cluster_1_pitch
- removed joint back_right__cluster_1_roll
- removed joint back_right__cluster_2_base_fix
- removed joint back_right__cluster_2_end_joint
- removed joint back_right__cluster_2_pitch
- removed joint back_right__cluster_2_roll
- removed joint back_right__cluster_3_base_fix
- removed joint back_right__cluster_3_end_joint
- removed joint back_right__cluster_3_mid_joint
- removed joint back_right__cluster_3_pitch
- removed joint back_right__cluster_3_roll
- removed joint back_right__cluster_3_wrist
- removed joint back_right__cluster_3_wrist_link_foot_joint
- removed joint base_joint
- removed joint base_link_back__sensor_joint
- removed joint base_link_back_left__joint
- removed joint base_link_back_right__joint
- removed joint base_link_front_left__joint
- removed joint base_link_front_left__sensor_joint
- removed joint base_link_front_right__joint
- removed joint base_link_front_right__sensor_joint
- removed joint base_link_left__sensor_joint
- removed joint base_link_right__sensor_joint
- removed joint bottom_lidar_base_joint
- removed joint front_left__cluster_1_base_fix
- removed joint front_left__cluster_1_end_joint
- removed joint front_left__cluster_1_pitch
- removed joint front_left__cluster_1_roll
- removed joint front_left__cluster_2_base_fix
- removed joint front_left__cluster_2_end_joint
- removed joint front_left__cluster_2_pitch
- removed joint front_left__cluster_2_roll
- removed joint front_left__cluster_3_base_fix
- removed joint front_left__cluster_3_end_joint
- removed joint front_left__cluster_3_mid_joint
- removed joint front_left__cluster_3_pitch
- removed joint front_left__cluster_3_roll
- removed joint front_left__cluster_3_wrist
- removed joint front_left__cluster_3_wrist_link_foot_joint
- removed joint front_right__cluster_1_base_fix
- removed joint front_right__cluster_1_end_joint
- removed joint front_right__cluster_1_pitch
- removed joint front_right__cluster_1_roll
- removed joint front_right__cluster_2_base_fix
- removed joint front_right__cluster_2_end_joint
- removed joint front_right__cluster_2_pitch
- removed joint front_right__cluster_2_roll
- removed joint front_right__cluster_3_base_fix
- removed joint front_right__cluster_3_end_joint
- removed joint front_right__cluster_3_mid_joint
- removed joint front_right__cluster_3_pitch
- removed joint front_right__cluster_3_roll
- removed joint front_right__cluster_3_wrist
- removed joint front_right__cluster_3_wrist_link_foot_joint
- removed joint top_lidar_base_joint
- added joint arm1_foot_link_joint: type fixed, parent arm1_link7, child arm1_foot_link, origin xyz=0.03 0 0 rpy=0 1.57 0
- added joint arm1_j1: type revolute, parent base_link, child arm1_link1, origin xyz=0.127 -0.1778 0 rpy=1.5707963267949 0 0, axis 1 0 0, limit lower=-3.14 upper=3.14 effort=10 velocity=10
- added joint arm1_j2: type revolute, parent arm1_link1, child arm1_link2, origin xyz=0.057944 0.00079375 0.0381 rpy=0 0 0, axis 0 1 0, limit lower=-3.14 upper=0.174 effort=10 velocity=10
- added joint arm1_j3: type revolute, parent arm1_link2, child arm1_link3, origin xyz=0.0547687500000001 0.000793750000000008 -0.03175 rpy=0 0 0, axis 1 0 0, limit lower=-3.14 upper=3.14 effort=10 velocity=10
- added joint arm1_j4: type revolute, parent arm1_link3, child arm1_link4, origin xyz=0.090483750066 0.000793749999999904 0.03175 rpy=0 0 0, axis 0 1 0, limit lower=-3.14 upper=0.174 effort=10 velocity=10
- added joint arm1_j5: type revolute, parent arm1_link4, child arm1_link5, origin xyz=0.0420687499999999 0.000793750000000015 -0.03175 rpy=0 0 0, axis 1 0 0, limit lower=-3.14 upper=3.14 effort=10 velocity=10
- added joint arm1_j6: type revolute, parent arm1_link5, child arm1_link6, origin xyz=0.10239 0.00079375 0.0254 rpy=0 0 0, axis 0 1 0, limit lower=-3.14 upper=0.174 effort=10 velocity=10
- added joint arm1_j7: type revolute, parent arm1_link6, child arm1_link7, origin xyz=0.0357187500000001 0.000793749999999943 -0.01905 rpy=0 0 0, axis 1 0 0, limit lower=-3.14 upper=3.14 effort=10 velocity=10
- added joint arm2_foot_link_joint: type fixed, parent arm2_link7, child arm2_foot_link, origin xyz=0.03 0 0 rpy=0 1.57 0
- added joint arm2_j1: type revolute, parent base_link, child arm2_link1, origin xyz=0.127 0.1778 0 rpy=1.5707963267949 0 0, axis 1 0 0, limit lower=-3.14 upper=3.14 effort=10 velocity=10
- added joint arm2_j2: type revolute, parent arm2_link1, child arm2_link2, origin xyz=0.057944 -0.00079375 -0.0381 rpy=0 0 0, axis 0 -1 0, limit lower=-3.14 upper=0.174 effort=10 velocity=10
- added joint arm2_j3: type revolute, parent arm2_link2, child arm2_link3, origin xyz=0.0547687500000002 -0.000793749999999992 0.03175 rpy=0 0 0, axis 1 0 0, limit lower=-3.14 upper=3.14 effort=10 velocity=10
- added joint arm2_j4: type revolute, parent arm2_link3, child arm2_link4, origin xyz=0.090484 -0.00079375 -0.03175 rpy=0 0 0, axis 0 -1 0, limit lower=-3.14 upper=0.174 effort=10 velocity=10
- added joint arm2_j5: type revolute, parent arm2_link4, child arm2_link5, origin xyz=0.0420687499999999 -0.000793750000000003 0.03175 rpy=0 0 0, axis 1 0 0, limit lower=-3.14 upper=3.14 effort=10 velocity=10
- added joint arm2_j6: type revolute, parent arm2_link5, child arm2_link6, origin xyz=0.10239 -0.00079375 -0.0254 rpy=0 0 0, axis 0 -1 0, limit lower=-3.14 upper=0.174 effort=10 velocity=10
- added joint arm2_j7: type revolute, parent arm2_link6, child arm2_link7, origin xyz=0.03571875 -0.000793749999999932 0.01905 rpy=0 0 0, axis 1 0 0, limit lower=-3.14 upper=3.14 effort=10 velocity=10
- added joint arm3_foot_link_joint: type fixed, parent arm3_link7, child arm3_foot_link, origin xyz=-0.03 0 0 rpy=0 1.57 0
- added joint arm3_j1: type revolute, parent base_link, child arm3_link1, origin xyz=-0.127 0.1778 0 rpy=1.5707963267949 0 0, axis -1 0 0, limit lower=-3.14 upper=3.14 effort=10 velocity=10
- added joint arm3_j2: type revolute, parent arm3_link1, child arm3_link2, origin xyz=-0.057944 0.00079375 -0.0381 rpy=0 0 0, axis 0 1 0, limit lower=-3.14 upper=0.174 effort=10 velocity=10
- added joint arm3_j3: type revolute, parent arm3_link2, child arm3_link3, origin xyz=-0.0547687500000001 0.000793750000000006 0.03175 rpy=0 0 0, axis -1 0 0, limit lower=-3.14 upper=3.14 effort=10 velocity=10
- added joint arm3_j4: type revolute, parent arm3_link3, child arm3_link4, origin xyz=-0.090484 0.00079375 -0.03175 rpy=0 0 0, axis 0 1 0, limit lower=-3.14 upper=0.174 effort=10 velocity=10
- added joint arm3_j5: type revolute, parent arm3_link4, child arm3_link5, origin xyz=-0.04206875 0.000793750000000013 0.03175 rpy=0 0 0, axis -1 0 0, limit lower=-3.14 upper=3.14 effort=10 velocity=10
- added joint arm3_j6: type revolute, parent arm3_link5, child arm3_link6, origin xyz=-0.10239 0.00079375 -0.0254 rpy=0 0 0, axis 0 1 0, limit lower=-3.14 upper=0.174 effort=10 velocity=10
- added joint arm3_j7: type revolute, parent arm3_link6, child arm3_link7, origin xyz=-0.03571875 0.000793749999999942 0.01905 rpy=0 0 0, axis -1 0 0, limit lower=-3.14 upper=3.14 effort=10 velocity=10
- added joint arm4_foot_link_joint: type fixed, parent arm4_link7, child arm4_foot_link, origin xyz=-0.03 0 0 rpy=0 1.57 0
- added joint arm4_j1: type revolute, parent base_link, child arm4_link1, origin xyz=-0.127 -0.1778 0 rpy=1.5707963267949 0 0, axis -1 0 0, limit lower=-3.14 upper=3.14 effort=10 velocity=10
- added joint arm4_j2: type revolute, parent arm4_link1, child arm4_link2, origin xyz=-0.057944 -0.00079375 0.0381 rpy=0 0 0, axis 0 -1 0, limit lower=-3.14 upper=0.174 effort=10 velocity=10
- added joint arm4_j3: type revolute, parent arm4_link2, child arm4_link3, origin xyz=-0.0547687500000001 -0.000793750000000011 -0.03175 rpy=0 0 0, axis -1 0 0, limit lower=-3.14 upper=3.14 effort=10 velocity=10
- added joint arm4_j4: type revolute, parent arm4_link3, child arm4_link4, origin xyz=-0.090484 -0.00079375 0.03175 rpy=0 0 0, axis 0 -1 0, limit lower=-3.14 upper=0.174 effort=10 velocity=10
- added joint arm4_j5: type revolute, parent arm4_link4, child arm4_link5, origin xyz=-0.0420687499999999 -0.000793750000000018 -0.03175 rpy=0 0 0, axis -1 0 0, limit lower=-3.14 upper=3.14 effort=10 velocity=10
- added joint arm4_j6: type revolute, parent arm4_link5, child arm4_link6, origin xyz=-0.10239 -0.00079375 0.0254 rpy=0 0 0, axis 0 -1 0, limit lower=-3.14 upper=0.174 effort=10 velocity=10
- added joint arm4_j7: type revolute, parent arm4_link6, child arm4_link7, origin xyz=-0.03571875 -0.000793749999999946 -0.01905 rpy=0 0 0, axis -1 0 0, limit lower=-3.14 upper=3.14 effort=10 velocity=10
- added joint back_sensor_link_joint: type fixed, parent base_link, child back_sensor_link, origin xyz=-0.28 0 -0.01 rpy=0 0 0
- added joint front_sensor_link_joint: type fixed, parent base_link, child front_sensor_link, origin xyz=0.28 0 -0.01 rpy=0 0 0

Commit message: Update joint gains to kp=20 kd=5

File: crab.urdf (robot description, URDF)
Before this commit: robot CRAB_Model_Assembly, 35 links, 34 joints
Links:
- link arm1_link1: geometry visual mesh filename=meshes/arm1_link1.STL
- link arm1_link2: geometry collision cylinder length=0.05 radius=0.04; visual mesh filename=meshes/arm1_link2.STL
- link arm1_link3: geometry collision cylinder length=0.05 radius=0.03; visual mesh filename=meshes/arm1_link3.STL
- link arm1_link4: geometry collision cylinder length=0.05 radius=0.03; visual mesh filename=meshes/arm1_link4.STL
- link arm1_link5: geometry collision cylinder length=0.07 radius=0.025; visual mesh filename=meshes/arm1_link5.STL
- link arm1_link6: geometry collision cylinder length=0.05 radius=0.02; visual mesh filename=meshes/arm1_link6.STL
- link arm1_link7: geometry visual mesh filename=meshes/arm1_link7.STL
- link arm2_link1: geometry visual mesh filename=meshes/arm2_link1.STL
- link arm2_link2: geometry collision cylinder length=0.05 radius=0.04; visual mesh filename=meshes/arm2_link2.STL
- link arm2_link3: geometry collision cylinder length=0.05 radius=0.03; visual mesh filename=meshes/arm2_link3.STL
- link arm2_link4: geometry collision cylinder length=0.05 radius=0.03; visual mesh filename=meshes/arm2_link4.STL
- link arm2_link5: geometry collision cylinder length=0.07 radius=0.025; visual mesh filename=meshes/arm2_link5.STL
- link arm2_link6: geometry collision cylinder length=0.05 radius=0.02; visual mesh filename=meshes/arm2_link6.STL
- link arm2_link7: geometry visual mesh filename=meshes/arm2_link7.STL
- link arm3_link1: geometry visual mesh filename=meshes/arm3_link1.STL
- link arm3_link2: geometry collision cylinder length=0.05 radius=0.04; visual mesh filename=meshes/arm3_link2.STL
- link arm3_link3: geometry collision cylinder length=0.05 radius=0.03; visual mesh filename=meshes/arm3_link3.STL
- link arm3_link4: geometry collision cylinder length=0.05 radius=0.03; visual mesh filename=meshes/arm3_link4.STL
- link arm3_link5: geometry collision cylinder length=0.07 radius=0.025; visual mesh filename=meshes/arm3_link5.STL
- link arm3_link6: geometry collision cylinder length=0.05 radius=0.02; visual mesh filename=meshes/arm3_link6.STL
- link arm3_link7: geometry visual mesh filename=meshes/arm3_link7.STL
- link arm4_link1: geometry visual mesh filename=meshes/arm4_link1.STL
- link arm4_link2: geometry collision cylinder length=0.05 radius=0.04; visual mesh filename=meshes/arm4_link2.STL
- link arm4_link3: geometry collision cylinder length=0.05 radius=0.03; visual mesh filename=meshes/arm4_link3.STL
- link arm4_link4: geometry collision cylinder length=0.05 radius=0.03; visual mesh filename=meshes/arm4_link4.STL
- link arm4_link5: geometry collision cylinder length=0.07 radius=0.025; visual mesh filename=meshes/arm4_link5.STL
- link arm4_link6: geometry collision cylinder length=0.05 radius=0.02; visual mesh filename=meshes/arm4_link6.STL
- link arm4_link7: geometry visual mesh filename=meshes/arm4_link7.STL
- link base_link: geometry collision box size=0.4 0.4 0.15; visual mesh filename=meshes/base_link.STL

Commit message: Change joint drive to force (for implicit actuators)

File: crab.urdf (robot description, URDF)
Before this commit: robot CRAB_Model_Assembly, 35 links, 34 joints
Links:
- link arm1_foot_link: mass 1e-10 -> 0.1
- link arm2_foot_link: mass 1e-10 -> 0.1
- link arm3_foot_link: mass 1e-10 -> 0.1
- link arm4_foot_link: mass 1e-10 -> 0.1
