Commit message: Adjust joint vel and effort limits

File: crab.urdf (robot description, URDF)
Before this commit: robot CRAB_Model_Assembly, 35 links, 34 joints
Joints:
- joint arm1_j1: limit lower=-3.14 upper=3.14 effort=10 velocity=10 -> lower=-3.14 upper=3.14 effort=300 velocity=100
- joint arm1_j2: limit lower=-3.14 upper=0.174 effort=10 velocity=10 -> lower=-3.14 upper=0.174 effort=300 velocity=100
- joint arm1_j3: limit lower=-3.14 upper=3.14 effort=10 velocity=10 -> lower=-3.14 upper=3.14 effort=300 velocity=100
- joint arm1_j4: limit lower=-3.14 upper=0.174 effort=10 velocity=10 -> lower=-3.14 upper=0.174 effort=300 velocity=100
- joint arm1_j5: limit lower=-3.14 upper=3.14 effort=10 velocity=10 -> lower=-3.14 upper=3.14 effort=300 velocity=100
- joint arm1_j6: limit lower=-3.14 upper=0.174 effort=10 velocity=10 -> lower=-3.14 upper=0.174 effort=300 velocity=100
- joint arm1_j7: limit lower=-3.14 upper=3.14 effort=10 velocity=10 -> lower=-3.14 upper=3.14 effort=300 velocity=100
- joint arm2_j1: limit lower=-3.14 upper=3.14 effort=10 velocity=10 -> lower=-3.14 upper=3.14 effort=300 velocity=100
- joint arm2_j2: limit lower=-3.14 upper=0.174 effort=10 velocity=10 -> lower=-3.14 upper=0.174 effort=300 velocity=100
- joint arm2_j3: limit lower=-3.14 upper=3.14 effort=10 velocity=10 -> lower=-3.14 upper=3.14 effort=300 velocity=100
- joint arm2_j4: limit lower=-3.14 upper=0.174 effort=10 velocity=10 -> lower=-3.14 upper=0.174 effort=300 velocity=100
- joint arm2_j5: limit lower=-3.14 upper=3.14 effort=10 velocity=10 -> lower=-3.14 upper=3.14 effort=300 velocity=100
- joint arm2_j6: limit lower=-3.14 upper=0.174 effort=10 velocity=10 -> lower=-3.14 upper=0.174 effort=300 velocity=100
- joint arm2_j7: limit lower=-3.14 upper=3.14 effort=10 velocity=10 -> lower=-3.14 upper=3.14 effort=300 velocity=100
- joint arm3_j1: limit lower=-3.14 upper=3.14 effort=10 velocity=10 -> lower=-3.14 upper=3.14 effort=300 velocity=100
- joint arm3_j2: limit lower=-3.14 upper=0.174 effort=10 velocity=10 -> lower=-3.14 upper=0.174 effort=300 velocity=100
- joint arm3_j3: limit lower=-3.14 upper=3.14 effort=10 velocity=10 -> lower=-3.14 upper=3.14 effort=300 velocity=100
- joint arm3_j4: limit lower=-3.14 upper=0.174 effort=10 velocity=10 -> lower=-3.14 upper=0.174 effort=300 velocity=100
- joint arm3_j5: limit lower=-3.14 upper=3.14 effort=10 velocity=10 -> lower=-3.14 upper=3.14 effort=300 velocity=100
- joint arm3_j6: limit lower=-3.14 upper=0.174 effort=10 velocity=10 -> lower=-3.14 upper=0.174 effort=300 velocity=100
- joint arm3_j7: limit lower=-3.14 upper=3.14 effort=10 velocity=10 -> lower=-3.14 upper=3.14 effort=300 velocity=100
- joint arm4_j1: limit lower=-3.14 upper=3.14 effort=10 velocity=10 -> lower=-3.14 upper=3.14 effort=300 velocity=100
- joint arm4_j2: limit lower=-3.14 upper=0.174 effort=10 velocity=10 -> lower=-3.14 upper=0.174 effort=300 velocity=100
- joint arm4_j3: limit lower=-3.14 upper=3.14 effort=10 velocity=10 -> lower=-3.14 upper=3.14 effort=300 velocity=100
- joint arm4_j4: limit lower=-3.14 upper=0.174 effort=10 velocity=10 -> lower=-3.14 upper=0.174 effort=300 velocity=100
- joint arm4_j5: limit lower=-3.14 upper=3.14 effort=10 velocity=10 -> lower=-3.14 upper=3.14 effort=300 velocity=100
- joint arm4_j6: limit lower=-3.14 upper=0.174 effort=10 velocity=10 -> lower=-3.14 upper=0.174 effort=300 velocity=100
- joint arm4_j7: limit lower=-3.14 upper=3.14 effort=10 velocity=10 -> lower=-3.14 upper=3.14 effort=300 velocity=100

Commit message: Modify URDF for body/leg contact termination

File: crab.urdf (robot description, URDF)
Before this commit: robot CRAB_Model_Assembly, 35 links, 34 joints
Links:
- link arm1_link2: geometry visual mesh filename=meshes/arm1_link2.STL
- link arm1_link3: geometry visual mesh filename=meshes/arm1_link3.STL
- link arm1_link4: geometry collision cylinder length=0.095 radius=0.0325; visual mesh filename=meshes/arm1_link4.STL
- link arm1_link6: geometry collision cylinder length=0.075 radius=0.025; visual mesh filename=meshes/arm1_link6.STL
- link arm2_link2: geometry visual mesh filename=meshes/arm2_link2.STL
- link arm2_link3: geometry visual mesh filename=meshes/arm2_link3.STL
- link arm2_link4: geometry collision cylinder length=0.095 radius=0.0325; visual mesh filename=meshes/arm2_link4.STL
- link arm2_link6: geometry collision cylinder length=0.075 radius=0.025; visual mesh filename=meshes/arm2_link6.STL
- link arm3_link2: geometry visual mesh filename=meshes/arm3_link2.STL
- link arm3_link3: geometry visual mesh filename=meshes/arm3_link3.STL
- link arm3_link4: geometry collision cylinder length=0.095 radius=0.0325; visual mesh filename=meshes/arm3_link4.STL
- link arm3_link6: geometry collision cylinder length=0.075 radius=0.025; visual mesh filename=meshes/arm3_link6.STL
- link arm4_link2: geometry visual mesh filename=meshes/arm4_link2.STL
- link arm4_link3: geometry visual mesh filename=meshes/arm4_link3.STL
- link arm4_link4: geometry collision cylinder length=0.095 radius=0.0325; visual mesh filename=meshes/arm4_link4.STL
- link arm4_link6: geometry collision cylinder length=0.075 radius=0.025; visual mesh filename=meshes/arm4_link6.STL
- link base_link: geometry collision cylinder length=0.17 radius=0.28; visual mesh filename=meshes/base_link.STL

Commit message: Revert "Adjust joint vel and effort limits"
This reverts commit a2973d8448791546b471ca00983f55674512c95b.

File: crab.urdf (robot description, URDF)
Before this commit: robot CRAB_Model_Assembly, 35 links, 34 joints
Joints:
- joint arm1_j1: limit lower=-3.14 upper=3.14 effort=300 velocity=100 -> lower=-3.14 upper=3.14 effort=10 velocity=10
- joint arm1_j2: limit lower=-3.14 upper=0.174 effort=300 velocity=100 -> lower=-3.14 upper=0.174 effort=10 velocity=10
- joint arm1_j3: limit lower=-3.14 upper=3.14 effort=300 velocity=100 -> lower=-3.14 upper=3.14 effort=10 velocity=10
- joint arm1_j4: limit lower=-3.14 upper=0.174 effort=300 velocity=100 -> lower=-3.14 upper=0.174 effort=10 velocity=10
- joint arm1_j5: limit lower=-3.14 upper=3.14 effort=300 velocity=100 -> lower=-3.14 upper=3.14 effort=10 velocity=10
- joint arm1_j6: limit lower=-3.14 upper=0.174 effort=300 velocity=100 -> lower=-3.14 upper=0.174 effort=10 velocity=10
- joint arm1_j7: limit lower=-3.14 upper=3.14 effort=300 velocity=100 -> lower=-3.14 upper=3.14 effort=10 velocity=10
- joint arm2_j1: limit lower=-3.14 upper=3.14 effort=300 velocity=100 -> lower=-3.14 upper=3.14 effort=10 velocity=10
- joint arm2_j2: limit lower=-3.14 upper=0.174 effort=300 velocity=100 -> lower=-3.14 upper=0.174 effort=10 velocity=10
- joint arm2_j3: limit lower=-3.14 upper=3.14 effort=300 velocity=100 -> lower=-3.14 upper=3.14 effort=10 velocity=10
- joint arm2_j4: limit lower=-3.14 upper=0.174 effort=300 velocity=100 -> lower=-3.14 upper=0.174 effort=10 velocity=10
- joint arm2_j5: limit lower=-3.14 upper=3.14 effort=300 velocity=100 -> lower=-3.14 upper=3.14 effort=10 velocity=10
- joint arm2_j6: limit lower=-3.14 upper=0.174 effort=300 velocity=100 -> lower=-3.14 upper=0.174 effort=10 velocity=10
- joint arm2_j7: limit lower=-3.14 upper=3.14 effort=300 velocity=100 -> lower=-3.14 upper=3.14 effort=10 velocity=10
- joint arm3_j1: limit lower=-3.14 upper=3.14 effort=300 velocity=100 -> lower=-3.14 upper=3.14 effort=10 velocity=10
- joint arm3_j2: limit lower=-3.14 upper=0.174 effort=300 velocity=100 -> lower=-3.14 upper=0.174 effort=10 velocity=10
- joint arm3_j3: limit lower=-3.14 upper=3.14 effort=300 velocity=100 -> lower=-3.14 upper=3.14 effort=10 velocity=10
- joint arm3_j4: limit lower=-3.14 upper=0.174 effort=300 velocity=100 -> lower=-3.14 upper=0.174 effort=10 velocity=10
- joint arm3_j5: limit lower=-3.14 upper=3.14 effort=300 velocity=100 -> lower=-3.14 upper=3.14 effort=10 velocity=10
- joint arm3_j6: limit lower=-3.14 upper=0.174 effort=300 velocity=100 -> lower=-3.14 upper=0.174 effort=10 velocity=10
- joint arm3_j7: limit lower=-3.14 upper=3.14 effort=300 velocity=100 -> lower=-3.14 upper=3.14 effort=10 velocity=10
- joint arm4_j1: limit lower=-3.14 upper=3.14 effort=300 velocity=100 -> lower=-3.14 upper=3.14 effort=10 velocity=10
- joint arm4_j2: limit lower=-3.14 upper=0.174 effort=300 velocity=100 -> lower=-3.14 upper=0.174 effort=10 velocity=10
- joint arm4_j3: limit lower=-3.14 upper=3.14 effort=300 velocity=100 -> lower=-3.14 upper=3.14 effort=10 velocity=10
- joint arm4_j4: limit lower=-3.14 upper=0.174 effort=300 velocity=100 -> lower=-3.14 upper=0.174 effort=10 velocity=10
- joint arm4_j5: limit lower=-3.14 upper=3.14 effort=300 velocity=100 -> lower=-3.14 upper=3.14 effort=10 velocity=10
- joint arm4_j6: limit lower=-3.14 upper=0.174 effort=300 velocity=100 -> lower=-3.14 upper=0.174 effort=10 velocity=10
- joint arm4_j7: limit lower=-3.14 upper=3.14 effort=300 velocity=100 -> lower=-3.14 upper=3.14 effort=10 velocity=10

Commit message: Add realistic crab with simplified collision meshes

File: crab.urdf (robot description, URDF)
Before this commit: robot CRAB_Model_Assembly, 35 links, 34 joints
Links:
- removed link back_sensor_link
- removed link front_sensor_link
- link arm1_foot_link: mass 0.1 -> 0.014479166215211; geometry collision sphere radius=0.023; visual mesh filename=meshes/arm1_link8.STL
- link arm1_link2: mass 0.792615281561028 -> 0.792615281561027; geometry visual mesh filename=meshes/arm1_link2.STL
- link arm1_link3: mass 0.914578646343626 -> 0.914578646343627; geometry visual mesh filename=meshes/arm1_link3.STL
- link arm1_link4: geometry collision cylinder length=0.0825 radius=0.035; visual mesh filename=meshes/arm1_link4.STL
- link arm1_link5: mass 0.632159217766391 -> 0.632159217766392
- link arm1_link6: geometry collision cylinder length=0.06 radius=0.025; visual mesh filename=meshes/arm1_link6.STL
- link arm2_foot_link: mass 0.1 -> 0.014479166215211; geometry collision sphere radius=0.023; visual mesh filename=meshes/arm2_link8.STL
- link arm2_link1: mass 0.935223157536645 -> 0.935223157536646
- link arm2_link2: mass 0.792615281561028 -> 0.792615281561027; geometry visual mesh filename=meshes/arm2_link2.STL
- link arm2_link3: geometry visual mesh filename=meshes/arm2_link3.STL
- link arm2_link4: geometry collision cylinder length=0.0825 radius=0.035; visual mesh filename=meshes/arm2_link4.STL
- link arm2_link5: mass 0.632159217766392 -> 0.632159217766391
- link arm2_link6: mass 0.174644982031482 -> 0.174644981799895; geometry collision cylinder length=0.06 radius=0.025; visual mesh filename=meshes/arm2_link6.STL
- link arm3_foot_link: mass 0.1 -> 0.014479166215211; geometry collision sphere radius=0.023; visual mesh filename=meshes/arm3_link8.STL
- link arm3_link1: mass 0.935223157536645 -> 0.935223157536646
- link arm3_link2: geometry visual mesh filename=meshes/arm3_link2.STL
- link arm3_link3: mass 0.914578646343627 -> 0.914578646343626; geometry visual mesh filename=meshes/arm3_link3.STL
- link arm3_link4: geometry collision cylinder length=0.0825 radius=0.035; visual mesh filename=meshes/arm3_link4.STL
- link arm3_link6: geometry collision cylinder length=0.06 radius=0.025; visual mesh filename=meshes/arm3_link6.STL
- link arm4_foot_link: mass 0.1 -> 0.014479166215211; geometry collision sphere radius=0.023; visual mesh filename=meshes/arm4_link8.STL
- link arm4_link2: geometry visual mesh filename=meshes/arm4_link2.STL
- link arm4_link3: mass 0.914578646343627 -> 0.914578646343626; geometry visual mesh filename=meshes/arm4_link3.STL
- link arm4_link4: geometry collision cylinder length=0.0825 radius=0.035; visual mesh filename=meshes/arm4_link4.STL
- link arm4_link5: mass 0.63215921776639 -> 0.632159217766391
- link arm4_link6: geometry collision cylinder length=0.06 radius=0.025; visual mesh filename=meshes/arm4_link6.STL
- link base_link: mass 11.6672712209699 -> 11.6672712209698; geometry collision cylinder length=0.2 radius=0.28; visual mesh filename=meshes/base_link.STL
Joints:
- removed joint arm1_foot_link_joint
- removed joint arm2_foot_link_joint
- removed joint arm3_foot_link_joint
- removed joint arm4_foot_link_joint
- removed joint back_sensor_link_joint
- removed joint front_sensor_link_joint
- added joint arm1_j8: type fixed, parent arm1_link7, child arm1_foot_link, origin xyz=0.01161 0 0 rpy=0 1.5708 0
- added joint arm2_j8: type fixed, parent arm2_link7, child arm2_foot_link, origin xyz=0.01161 0 0 rpy=0 1.5708 0
- added joint arm3_j8: type fixed, parent arm3_link7, child arm3_foot_link, origin xyz=-0.01161 0 0 rpy=0 1.5708 0
- added joint arm4_j8: type fixed, parent arm4_link7, child arm4_foot_link, origin xyz=-0.01161 0 0 rpy=0 1.5708 0
- joint arm1_j2: axis 0 1 0 -> 0 -1 0; origin xyz=0.057944 0.00079375 0.0381 rpy=0 0 0 -> xyz=0.05794375 0.000793749999999943 0.0381000000000001 rpy=0 0 0
- joint arm1_j6: axis 0 1 0 -> 0 -1 0; origin xyz=0.10239 0.00079375 0.0254 rpy=0 0 0 -> xyz=0.10239375 0.000793749999999789 0.0254 rpy=0 0 0
- joint arm2_j1: origin xyz=0.127 0.1778 0 rpy=1.5707963267949 0 0 -> xyz=0.127 0.1778 0 rpy=1.5708 0 0
- joint arm2_j2: axis 0 -1 0 -> 0 1 0; origin xyz=0.057944 -0.00079375 -0.0381 rpy=0 0 0 -> xyz=0.05794375 -0.000793749999999922 -0.0381000000000001 rpy=0 0 0
- joint arm2_j4: origin xyz=0.090484 -0.00079375 -0.03175 rpy=0 0 0 -> xyz=0.090483750066 -0.000793749999999871 -0.0317500000000001 rpy=0 0 0
- joint arm2_j6: axis 0 -1 0 -> 0 1 0; origin xyz=0.10239 -0.00079375 -0.0254 rpy=0 0 0 -> xyz=0.10239375 -0.000793749999999754 -0.0254000000000001 rpy=0 0 0
- joint arm3_j1: origin xyz=-0.127 0.1778 0 rpy=1.5707963267949 0 0 -> xyz=-0.127 0.1778 0 rpy=1.5708 0 0
- joint arm3_j2: axis 0 1 0 -> 0 -1 0; origin xyz=-0.057944 0.00079375 -0.0381 rpy=0 0 0 -> xyz=-0.05794375 0.000793750000000014 -0.0381000000000001 rpy=0 0 0
- joint arm3_j4: origin xyz=-0.090484 0.00079375 -0.03175 rpy=0 0 0 -> xyz=-0.090483750066 0.000793749999999906 -0.03175 rpy=0 0 0
- joint arm3_j6: axis 0 1 0 -> 0 -1 0; origin xyz=-0.10239 0.00079375 -0.0254 rpy=0 0 0 -> xyz=-0.10239375 0.000793749999999791 -0.0254 rpy=0 0 0
- joint arm4_j2: axis 0 -1 0 -> 0 1 0; origin xyz=-0.057944 -0.00079375 0.0381 rpy=0 0 0 -> xyz=-0.0579437500000001 -0.000793749999999984 0.0381 rpy=0 0 0
- joint arm4_j4: origin xyz=-0.090484 -0.00079375 0.03175 rpy=0 0 0 -> xyz=-0.090483750066 -0.000793749999999901 0.03175 rpy=0 0 0
- joint arm4_j6: axis 0 -1 0 -> 0 1 0; origin xyz=-0.10239 -0.00079375 0.0254 rpy=0 0 0 -> xyz=-0.10239375 -0.000793749999999786 0.0254 rpy=0 0 0

Commit message: Scale foot link masses by 10

File: crab.urdf (robot description, URDF)
Before this commit: robot CRAB_Model_Assembly, 33 links, 32 joints
Links:
- link arm1_foot_link: mass 0.014479166215211 -> 0.14479166215211
- link arm2_foot_link: mass 0.014479166215211 -> 0.14479166215211
- link arm3_foot_link: mass 0.014479166215211 -> 0.14479166215211
- link arm4_foot_link: mass 0.014479166215211 -> 0.14479166215211

Commit message: Fix some joint position limits in URDF

File: crab.urdf (robot description, URDF)
Before this commit: robot CRAB_Model_Assembly, 33 links, 32 joints
Joints:
- joint arm1_j2: limit lower=-3.14 upper=0.174 effort=300 velocity=100 -> lower=-0.174 upper=3.14 effort=300 velocity=100
- joint arm1_j6: limit lower=-3.14 upper=0.174 effort=300 velocity=100 -> lower=-0.174 upper=3.14 effort=300 velocity=100
- joint arm2_j2: limit lower=-3.14 upper=0.174 effort=300 velocity=100 -> lower=-0.174 upper=3.14 effort=300 velocity=100
- joint arm2_j6: limit lower=-3.14 upper=0.174 effort=300 velocity=100 -> lower=-0.174 upper=3.14 effort=300 velocity=100
- joint arm3_j2: limit lower=-3.14 upper=0.174 effort=300 velocity=100 -> lower=-0.174 upper=3.14 effort=300 velocity=100
- joint arm3_j6: limit lower=-3.14 upper=0.174 effort=300 velocity=100 -> lower=-0.174 upper=3.14 effort=300 velocity=100
- joint arm4_j2: limit lower=-3.14 upper=0.174 effort=300 velocity=100 -> lower=-0.174 upper=3.14 effort=300 velocity=100
- joint arm4_j6: limit lower=-3.14 upper=0.174 effort=300 velocity=100 -> lower=-0.174 upper=3.14 effort=300 velocity=100

Commit message: Use simple base link collision mesh (instead of cylinder)

File: crab.urdf (robot description, URDF)
Before this commit: robot CRAB_Model_Assembly, 33 links, 32 joints
Links:
- link base_link: geometry collision mesh filename=meshes/base_link_collision.STL; visual mesh filename=meshes/base_link.STL
