Commit message: Clean up RSS urdf

File: rss/rss_new_base_arms.urdf (robot description, URDF)
Before this commit: robot combined_hexapods, 124 links, 122 joints
Links:
- removed link base_link
- removed link end_wall
- removed link far_wall
- removed link han_base
- removed link han_base_link
- removed link han_base_link_inertia
- removed link han_cable_harness_arm_link
- removed link han_cable_harness_ee_link
- removed link han_cable_harness_elbow_link
- removed link han_camera
- removed link han_camera_mount
- removed link han_finger_mount_left
- removed link han_finger_mount_right
- removed link han_flange
- removed link han_forearm_link
- removed link han_ft_frame
- removed link han_gripper_adapter
- removed link han_left_finger
- removed link han_mount_adapter
- removed link han_right_finger
- removed link han_shoulder_link
- removed link han_tool0
- removed link han_upper_arm_link
- removed link han_ur_mounting_frame
- removed link han_wrist_1_link
- removed link han_wrist_2_link
- removed link han_wrist_3_link
- removed link han_zimmer_body
- removed link han_zimmer_grasp_frame
- removed link metal_box_link
- removed link near_wall
- removed link slide_ati_ft_sensor
- removed link slide_ati_to_tombstone
- removed link slide_hexapod_home
- removed link slide_tombstone
- removed link ur20b_han_base
- removed link ur20b_han_base_link
- removed link ur20b_han_base_link_inertia
- removed link ur20b_han_cable_harness_arm_link
- removed link ur20b_han_cable_harness_ee_link
- removed link ur20b_han_cable_harness_elbow_link
- removed link ur20b_han_camera
- removed link ur20b_han_camera_mount
- removed link ur20b_han_finger_mount_left
- removed link ur20b_han_finger_mount_right
- removed link ur20b_han_flange
- removed link ur20b_han_forearm_link
- removed link ur20b_han_ft_frame
- removed link ur20b_han_gripper_adapter
- removed link ur20b_han_left_finger
- removed link ur20b_han_mount_adapter
- removed link ur20b_han_right_finger
- removed link ur20b_han_shoulder_link
- removed link ur20b_han_tool0
- removed link ur20b_han_upper_arm_link
- removed link ur20b_han_ur_mounting_frame
- removed link ur20b_han_wrist_1_link
- removed link ur20b_han_wrist_2_link
- removed link ur20b_han_wrist_3_link
- removed link ur20b_han_zimmer_body
- removed link ur20b_han_zimmer_grasp_frame
- removed link ur20b_slide_ati_ft_sensor
- removed link ur20b_slide_ati_to_tombstone
- removed link ur20b_slide_tombstone
- removed link ur20c_han_base
- removed link ur20c_han_base_link
- removed link ur20c_han_base_link_inertia
- removed link ur20c_han_cable_harness_arm_link
- removed link ur20c_han_cable_harness_ee_link
- removed link ur20c_han_cable_harness_elbow_link
- removed link ur20c_han_camera
- removed link ur20c_han_camera_mount
- removed link ur20c_han_finger_mount_left
- removed link ur20c_han_finger_mount_right
- removed link ur20c_han_flange
- removed link ur20c_han_forearm_link
- removed link ur20c_han_ft_frame
- removed link ur20c_han_gripper_adapter
- removed link ur20c_han_left_finger
- removed link ur20c_han_mount_adapter
- removed link ur20c_han_right_finger
- removed link ur20c_han_shoulder_link
- removed link ur20c_han_tool0
- removed link ur20c_han_upper_arm_link
- removed link ur20c_han_ur_mounting_frame
- removed link ur20c_han_wrist_1_link
- removed link ur20c_han_wrist_2_link
- removed link ur20c_han_wrist_3_link
- removed link ur20c_han_zimmer_body
- removed link ur20c_han_zimmer_grasp_frame
- removed link ur20c_slide_ati_ft_sensor
- removed link ur20c_slide_ati_to_tombstone
- removed link ur20c_slide_tombstone
- removed link ur20d_han_base
- removed link ur20d_han_base_link
- removed link ur20d_han_base_link_inertia
- removed link ur20d_han_cable_harness_arm_link
- removed link ur20d_han_cable_harness_ee_link
- removed link ur20d_han_cable_harness_elbow_link
- removed link ur20d_han_camera
- removed link ur20d_han_camera_mount
- removed link ur20d_han_finger_mount_left
- removed link ur20d_han_finger_mount_right
- removed link ur20d_han_flange
- removed link ur20d_han_forearm_link
- removed link ur20d_han_ft_frame
- removed link ur20d_han_gripper_adapter
- removed link ur20d_han_left_finger
- removed link ur20d_han_mount_adapter
- removed link ur20d_han_right_finger
- removed link ur20d_han_shoulder_link
- removed link ur20d_han_tool0
- removed link ur20d_han_upper_arm_link
- removed link ur20d_han_ur_mounting_frame
- removed link ur20d_han_wrist_1_link
- removed link ur20d_han_wrist_2_link
- removed link ur20d_han_wrist_3_link
- removed link ur20d_han_zimmer_body
- removed link ur20d_han_zimmer_grasp_frame
- removed link ur20d_slide_ati_ft_sensor
- removed link ur20d_slide_ati_to_tombstone
- removed link ur20d_slide_tombstone
- added link arm1_base_link; collision cylinder length=0.0254 radius=0.095; visual cylinder length=0.0254 radius=0.095
- added link arm1_cable_harness_arm_link; collision box size=0.07 0.1524 0.07; collision cylinder length=0.8 radius=0.0381
- added link arm1_cable_harness_ee_link; collision box size=0.1778 0.0762 0.0254; visual box size=0.1778 0.0762 0.0254
- added link arm1_cable_harness_elbow_link; collision box size=0.15 0.0762 0.15; visual box size=0.15 0.0762 0.15
- added link arm1_camera; collision mesh filename=meshes/rss_ur20/CAMERA.STL; visual mesh filename=meshes/rss_ur20/CAMERA_VISUAL_BASE.STL
- added link arm1_camera_mount; collision mesh filename=meshes/rss_ur20/CAMERA_MOUNT.STL; visual mesh filename=meshes/rss_ur20/CAMERA_MOUNT_VISUAL.STL
- added link arm1_finger1; collision mesh filename=meshes/rss_ur20/Finray_Finger.STL; visual mesh filename=meshes/rss_ur20/Finray_Finger.STL
- added link arm1_finger1_mount; collision mesh filename=meshes/zimmer_gripper_description/ZIMMER_SLIDE.STL; visual mesh filename=meshes/zimmer_gripper_description/ZIMMER_SLIDE.STL
- added link arm1_finger2; collision mesh filename=meshes/rss_ur20/Finray_Finger.STL; visual mesh filename=meshes/rss_ur20/Finray_Finger.STL
- added link arm1_finger2_mount; collision mesh filename=meshes/zimmer_gripper_description/ZIMMER_SLIDE.STL; visual mesh filename=meshes/zimmer_gripper_description/ZIMMER_SLIDE.STL
- added link arm1_gripper_adapter; collision mesh filename=meshes/rss_ur20/GRIPPER_PLATE.STL; visual mesh filename=meshes/rss_ur20/GRIPPER_PLATE_VISUAL.STL
- added link arm1_link1, mass 4.0; collision mesh filename=meshes/ur20/collision/base.stl; visual mesh filename=meshes/ur20/visual/base.dae
- added link arm1_link2, mass 16.343; collision mesh filename=meshes/ur20/collision/shoulder.stl; visual mesh filename=meshes/ur20/visual/shoulder.dae
- added link arm1_link3, mass 29.632; collision mesh filename=meshes/ur20/collision/upperarm.stl; visual mesh filename=meshes/ur20/visual/upperarm.dae
- added link arm1_link4, mass 7.879; collision mesh filename=meshes/ur20/collision/forearm.stl; visual mesh filename=meshes/ur20/visual/forearm.dae
- added link arm1_link5, mass 3.054; collision mesh filename=meshes/ur20/collision/wrist1.stl; visual mesh filename=meshes/ur20/visual/wrist1.dae
- added link arm1_link6, mass 3.126; collision mesh filename=meshes/ur20/collision/wrist2.stl; visual mesh filename=meshes/ur20/visual/wrist2.dae
- added link arm1_link7, mass 0.926; collision mesh filename=meshes/ur20/collision/wrist3.stl; visual mesh filename=meshes/ur20/visual/wrist3.dae
- added link arm1_mount_adapter; collision mesh filename=meshes/rss_ur20/MOUNT_PLATE.STL; visual mesh filename=meshes/rss_ur20/MOUNT_PLATE_VISUAL.STL
- added link arm1_slide_tombstone; collision box size=0.245 0.258 0.190; visual mesh filename=meshes/rss_ur20/tombstone.stl
- added link arm1_zimmer_body; collision mesh filename=meshes/zimmer_gripper_description/ZIMMER_BOX.STL; visual mesh filename=meshes/zimmer_gripper_description/ZIMMER_BOX.STL
- added link arm2_base_link; collision cylinder length=0.0254 radius=0.095; visual cylinder length=0.0254 radius=0.095
- added link arm2_cable_harness_arm_link; collision box size=0.07 0.1524 0.07; collision cylinder length=0.8 radius=0.0381
- added link arm2_cable_harness_ee_link; collision box size=0.1778 0.0762 0.0254; visual box size=0.1778 0.0762 0.0254
- added link arm2_cable_harness_elbow_link; collision box size=0.15 0.0762 0.15; visual box size=0.15 0.0762 0.15
- added link arm2_camera; collision mesh filename=meshes/rss_ur20/CAMERA.STL; visual mesh filename=meshes/rss_ur20/CAMERA_VISUAL_BASE.STL
- added link arm2_camera_mount; collision mesh filename=meshes/rss_ur20/CAMERA_MOUNT.STL; visual mesh filename=meshes/rss_ur20/CAMERA_MOUNT_VISUAL.STL
- added link arm2_finger1; collision mesh filename=meshes/rss_ur20/Finray_Finger.STL; visual mesh filename=meshes/rss_ur20/Finray_Finger.STL
- added link arm2_finger1_mount; collision mesh filename=meshes/zimmer_gripper_description/ZIMMER_SLIDE.STL; visual mesh filename=meshes/zimmer_gripper_description/ZIMMER_SLIDE.STL
- added link arm2_finger2; collision mesh filename=meshes/rss_ur20/Finray_Finger.STL; visual mesh filename=meshes/rss_ur20/Finray_Finger.STL
- added link arm2_finger2_mount; collision mesh filename=meshes/zimmer_gripper_description/ZIMMER_SLIDE.STL; visual mesh filename=meshes/zimmer_gripper_description/ZIMMER_SLIDE.STL
- added link arm2_gripper_adapter; collision mesh filename=meshes/rss_ur20/GRIPPER_PLATE.STL; visual mesh filename=meshes/rss_ur20/GRIPPER_PLATE_VISUAL.STL
- added link arm2_link1, mass 4.0; collision mesh filename=meshes/ur20/collision/base.stl; visual mesh filename=meshes/ur20/visual/base.dae
- added link arm2_link2, mass 16.343; collision mesh filename=meshes/ur20/collision/shoulder.stl; visual mesh filename=meshes/ur20/visual/shoulder.dae
- added link arm2_link3, mass 29.632; collision mesh filename=meshes/ur20/collision/upperarm.stl; visual mesh filename=meshes/ur20/visual/upperarm.dae
- added link arm2_link4, mass 7.879; collision mesh filename=meshes/ur20/collision/forearm.stl; visual mesh filename=meshes/ur20/visual/forearm.dae
- added link arm2_link5, mass 3.054; collision mesh filename=meshes/ur20/collision/wrist1.stl; visual mesh filename=meshes/ur20/visual/wrist1.dae
- added link arm2_link6, mass 3.126; collision mesh filename=meshes/ur20/collision/wrist2.stl; visual mesh filename=meshes/ur20/visual/wrist2.dae
- added link arm2_link7, mass 0.926; collision mesh filename=meshes/ur20/collision/wrist3.stl; visual mesh filename=meshes/ur20/visual/wrist3.dae
- added link arm2_mount_adapter; collision mesh filename=meshes/rss_ur20/MOUNT_PLATE.STL; visual mesh filename=meshes/rss_ur20/MOUNT_PLATE_VISUAL.STL
- added link arm2_slide_tombstone; collision box size=0.245 0.258 0.190; visual mesh filename=meshes/rss_ur20/tombstone.stl
- added link arm2_zimmer_body; collision mesh filename=meshes/zimmer_gripper_description/ZIMMER_BOX.STL; visual mesh filename=meshes/zimmer_gripper_description/ZIMMER_BOX.STL
- added link arm3_base_link; collision cylinder length=0.0254 radius=0.095; visual cylinder length=0.0254 radius=0.095
- added link arm3_cable_harness_arm_link; collision box size=0.07 0.1524 0.07; collision cylinder length=0.8 radius=0.0381
- added link arm3_cable_harness_ee_link; collision box size=0.1778 0.0762 0.0254; visual box size=0.1778 0.0762 0.0254
- added link arm3_cable_harness_elbow_link; collision box size=0.15 0.0762 0.15; visual box size=0.15 0.0762 0.15
- added link arm3_camera; collision mesh filename=meshes/rss_ur20/CAMERA.STL; visual mesh filename=meshes/rss_ur20/CAMERA_VISUAL_BASE.STL
- added link arm3_camera_mount; collision mesh filename=meshes/rss_ur20/CAMERA_MOUNT.STL; visual mesh filename=meshes/rss_ur20/CAMERA_MOUNT_VISUAL.STL
- added link arm3_finger1; collision mesh filename=meshes/rss_ur20/Finray_Finger.STL; visual mesh filename=meshes/rss_ur20/Finray_Finger.STL
- added link arm3_finger1_mount; collision mesh filename=meshes/zimmer_gripper_description/ZIMMER_SLIDE.STL; visual mesh filename=meshes/zimmer_gripper_description/ZIMMER_SLIDE.STL
- added link arm3_finger2; collision mesh filename=meshes/rss_ur20/Finray_Finger.STL; visual mesh filename=meshes/rss_ur20/Finray_Finger.STL
- added link arm3_finger2_mount; collision mesh filename=meshes/zimmer_gripper_description/ZIMMER_SLIDE.STL; visual mesh filename=meshes/zimmer_gripper_description/ZIMMER_SLIDE.STL
- added link arm3_gripper_adapter; collision mesh filename=meshes/rss_ur20/GRIPPER_PLATE.STL; visual mesh filename=meshes/rss_ur20/GRIPPER_PLATE_VISUAL.STL
- added link arm3_link1, mass 4.0; collision mesh filename=meshes/ur20/collision/base.stl; visual mesh filename=meshes/ur20/visual/base.dae
- added link arm3_link2, mass 16.343; collision mesh filename=meshes/ur20/collision/shoulder.stl; visual mesh filename=meshes/ur20/visual/shoulder.dae
- added link arm3_link3, mass 29.632; collision mesh filename=meshes/ur20/collision/upperarm.stl; visual mesh filename=meshes/ur20/visual/upperarm.dae
- added link arm3_link4, mass 7.879; collision mesh filename=meshes/ur20/collision/forearm.stl; visual mesh filename=meshes/ur20/visual/forearm.dae
- added link arm3_link5, mass 3.054; collision mesh filename=meshes/ur20/collision/wrist1.stl; visual mesh filename=meshes/ur20/visual/wrist1.dae
- added link arm3_link6, mass 3.126; collision mesh filename=meshes/ur20/collision/wrist2.stl; visual mesh filename=meshes/ur20/visual/wrist2.dae
- added link arm3_link7, mass 0.926; collision mesh filename=meshes/ur20/collision/wrist3.stl; visual mesh filename=meshes/ur20/visual/wrist3.dae
- added link arm3_mount_adapter; collision mesh filename=meshes/rss_ur20/MOUNT_PLATE.STL; visual mesh filename=meshes/rss_ur20/MOUNT_PLATE_VISUAL.STL
- added link arm3_slide_tombstone; collision box size=0.245 0.258 0.190; visual mesh filename=meshes/rss_ur20/tombstone.stl
- added link arm3_zimmer_body; collision mesh filename=meshes/zimmer_gripper_description/ZIMMER_BOX.STL; visual mesh filename=meshes/zimmer_gripper_description/ZIMMER_BOX.STL
- added link arm4_base_link; collision cylinder length=0.0254 radius=0.095; visual cylinder length=0.0254 radius=0.095
- added link arm4_cable_harness_arm_link; collision box size=0.07 0.1524 0.07; collision cylinder length=0.8 radius=0.0381
- added link arm4_cable_harness_ee_link; collision box size=0.1778 0.0762 0.0254; visual box size=0.1778 0.0762 0.0254
- added link arm4_cable_harness_elbow_link; collision box size=0.15 0.0762 0.15; visual box size=0.15 0.0762 0.15
- added link arm4_camera; collision mesh filename=meshes/rss_ur20/CAMERA.STL; visual mesh filename=meshes/rss_ur20/CAMERA_VISUAL_BASE.STL
- added link arm4_camera_mount; collision mesh filename=meshes/rss_ur20/CAMERA_MOUNT.STL; visual mesh filename=meshes/rss_ur20/CAMERA_MOUNT_VISUAL.STL
- added link arm4_finger1; collision mesh filename=meshes/rss_ur20/Finray_Finger.STL; visual mesh filename=meshes/rss_ur20/Finray_Finger.STL
- added link arm4_finger1_mount; collision mesh filename=meshes/zimmer_gripper_description/ZIMMER_SLIDE.STL; visual mesh filename=meshes/zimmer_gripper_description/ZIMMER_SLIDE.STL
- added link arm4_finger2; collision mesh filename=meshes/rss_ur20/Finray_Finger.STL; visual mesh filename=meshes/rss_ur20/Finray_Finger.STL
- added link arm4_finger2_mount; collision mesh filename=meshes/zimmer_gripper_description/ZIMMER_SLIDE.STL; visual mesh filename=meshes/zimmer_gripper_description/ZIMMER_SLIDE.STL
- added link arm4_gripper_adapter; collision mesh filename=meshes/rss_ur20/GRIPPER_PLATE.STL; visual mesh filename=meshes/rss_ur20/GRIPPER_PLATE_VISUAL.STL
- added link arm4_link1, mass 4.0; collision mesh filename=meshes/ur20/collision/base.stl; visual mesh filename=meshes/ur20/visual/base.dae
- added link arm4_link2, mass 16.343; collision mesh filename=meshes/ur20/collision/shoulder.stl; visual mesh filename=meshes/ur20/visual/shoulder.dae
- added link arm4_link3, mass 29.632; collision mesh filename=meshes/ur20/collision/upperarm.stl; visual mesh filename=meshes/ur20/visual/upperarm.dae
- added link arm4_link4, mass 7.879; collision mesh filename=meshes/ur20/collision/forearm.stl; visual mesh filename=meshes/ur20/visual/forearm.dae
- added link arm4_link5, mass 3.054; collision mesh filename=meshes/ur20/collision/wrist1.stl; visual mesh filename=meshes/ur20/visual/wrist1.dae
- added link arm4_link6, mass 3.126; collision mesh filename=meshes/ur20/collision/wrist2.stl; visual mesh filename=meshes/ur20/visual/wrist2.dae
- added link arm4_link7, mass 0.926; collision mesh filename=meshes/ur20/collision/wrist3.stl; visual mesh filename=meshes/ur20/visual/wrist3.dae
- added link arm4_mount_adapter; collision mesh filename=meshes/rss_ur20/MOUNT_PLATE.STL; visual mesh filename=meshes/rss_ur20/MOUNT_PLATE_VISUAL.STL
- added link arm4_slide_tombstone; collision box size=0.245 0.258 0.190; visual mesh filename=meshes/rss_ur20/tombstone.stl
- added link arm4_zimmer_body; collision mesh filename=meshes/zimmer_gripper_description/ZIMMER_BOX.STL; visual mesh filename=meshes/zimmer_gripper_description/ZIMMER_BOX.STL
Joints:
- removed joint base_link_to_end_wall
- removed joint base_link_to_far_wall
- removed joint base_link_to_metal_box
- removed joint base_link_to_near_wall
- removed joint gripper_adapter
- removed joint gripper_finger1_joint
- removed joint gripper_finger2_joint
- removed joint han_base_joint
- removed joint han_base_link-base_fixed_joint
- removed joint han_base_link-base_link_inertia
- removed joint han_cable_harness_arm_link
- removed joint han_cable_harness_ee_link
- removed joint han_cable_harness_elbow_link
- removed joint han_camera
- removed joint han_camera_mount
- removed joint han_elbow_joint
- removed joint han_flange-tool0
- removed joint han_left_finger
- removed joint han_mount_adapter
- removed joint han_right_finger
- removed joint han_shoulder_lift_joint
- removed joint han_shoulder_pan_joint
- removed joint han_ur_mounting_frame_joint
- removed joint han_wrist_1_joint
- removed joint han_wrist_2_joint
- removed joint han_wrist_3-flange
- removed joint han_wrist_3_joint
- removed joint han_wrist_3_link-ft_frame
- removed joint han_zimmer_body
- removed joint han_zimmer_grasp_frame_joint
- removed joint rotary_base_joint
- removed joint slide_ati_to_tombstone_joint
- removed joint slide_hex_joint
- removed joint slide_optical_plate_to_ur20_joint
- removed joint slide_optical_plate_to_ur20b_joint
- removed joint slide_optical_plate_to_ur20c_joint
- removed joint slide_optical_plate_to_ur20d_joint
- removed joint slide_tombstone_joint
- removed joint ur20b_gripper_adapter
- removed joint ur20b_gripper_finger1_joint
- removed joint ur20b_gripper_finger2_joint
- removed joint ur20b_han_base_joint
- removed joint ur20b_han_base_link-base_fixed_joint
- removed joint ur20b_han_base_link-base_link_inertia
- removed joint ur20b_han_cable_harness_arm_link
- removed joint ur20b_han_cable_harness_ee_link
- removed joint ur20b_han_cable_harness_elbow_link
- removed joint ur20b_han_camera
- removed joint ur20b_han_camera_mount
- removed joint ur20b_han_elbow_joint
- removed joint ur20b_han_flange-tool0
- removed joint ur20b_han_left_finger
- removed joint ur20b_han_mount_adapter
- removed joint ur20b_han_right_finger
- removed joint ur20b_han_shoulder_lift_joint
- removed joint ur20b_han_shoulder_pan_joint
- removed joint ur20b_han_ur_mounting_frame_joint
- removed joint ur20b_han_wrist_1_joint
- removed joint ur20b_han_wrist_2_joint
- removed joint ur20b_han_wrist_3-flange
- removed joint ur20b_han_wrist_3_joint
- removed joint ur20b_han_wrist_3_link-ft_frame
- removed joint ur20b_han_zimmer_body
- removed joint ur20b_han_zimmer_grasp_frame_joint
- removed joint ur20b_slide_ati_to_tombstone_joint
- removed joint ur20b_slide_tombstone_joint
- removed joint ur20c_gripper_adapter
- removed joint ur20c_gripper_finger1_joint
- removed joint ur20c_gripper_finger2_joint
- removed joint ur20c_han_base_joint
- removed joint ur20c_han_base_link-base_fixed_joint
- removed joint ur20c_han_base_link-base_link_inertia
- removed joint ur20c_han_cable_harness_arm_link
- removed joint ur20c_han_cable_harness_ee_link
- removed joint ur20c_han_cable_harness_elbow_link
- removed joint ur20c_han_camera
- removed joint ur20c_han_camera_mount
- removed joint ur20c_han_elbow_joint
- removed joint ur20c_han_flange-tool0
- removed joint ur20c_han_left_finger
- removed joint ur20c_han_mount_adapter
- removed joint ur20c_han_right_finger
- removed joint ur20c_han_shoulder_lift_joint
- removed joint ur20c_han_shoulder_pan_joint
- removed joint ur20c_han_ur_mounting_frame_joint
- removed joint ur20c_han_wrist_1_joint
- removed joint ur20c_han_wrist_2_joint
- removed joint ur20c_han_wrist_3-flange
- removed joint ur20c_han_wrist_3_joint
- removed joint ur20c_han_wrist_3_link-ft_frame
- removed joint ur20c_han_zimmer_body
- removed joint ur20c_han_zimmer_grasp_frame_joint
- removed joint ur20c_slide_ati_to_tombstone_joint
- removed joint ur20c_slide_tombstone_joint
- removed joint ur20d_gripper_adapter
- removed joint ur20d_gripper_finger1_joint
- removed joint ur20d_gripper_finger2_joint
- removed joint ur20d_han_base_joint
- removed joint ur20d_han_base_link-base_fixed_joint
- removed joint ur20d_han_base_link-base_link_inertia
- removed joint ur20d_han_cable_harness_arm_link
- removed joint ur20d_han_cable_harness_ee_link
- removed joint ur20d_han_cable_harness_elbow_link
- removed joint ur20d_han_camera
- removed joint ur20d_han_camera_mount
- removed joint ur20d_han_elbow_joint
- removed joint ur20d_han_flange-tool0
- removed joint ur20d_han_left_finger
- removed joint ur20d_han_mount_adapter
- removed joint ur20d_han_right_finger
- removed joint ur20d_han_shoulder_lift_joint
- removed joint ur20d_han_shoulder_pan_joint
- removed joint ur20d_han_ur_mounting_frame_joint
- removed joint ur20d_han_wrist_1_joint
- removed joint ur20d_han_wrist_2_joint
- removed joint ur20d_han_wrist_3-flange
- removed joint ur20d_han_wrist_3_joint
- removed joint ur20d_han_wrist_3_link-ft_frame
- removed joint ur20d_han_zimmer_body
- removed joint ur20d_han_zimmer_grasp_frame_joint
- removed joint ur20d_slide_ati_to_tombstone_joint
- removed joint ur20d_slide_tombstone_joint
- added joint arm1_adapter_joint: type fixed, parent arm1_link7, child arm1_mount_adapter, origin xyz=0 -0.00317 0 rpy=1.5707963 -1.5707963 0
- added joint arm1_base_joint: type fixed, parent arm1_slide_tombstone, child arm1_link1, origin xyz=0 0 0 rpy=0 0 0
- added joint arm1_cable_harness_arm_link: type fixed, parent arm1_link3, child arm1_cable_harness_arm_link, origin xyz=0 0 0 rpy=0 0 0
- added joint arm1_cable_harness_ee_link: type fixed, parent arm1_link7, child arm1_cable_harness_ee_link, origin xyz=0 0 0 rpy=0 0 0
- added joint arm1_cable_harness_elbow_link: type fixed, parent arm1_link4, child arm1_cable_harness_elbow_link, origin xyz=0 0 0 rpy=0 0 0
- added joint arm1_camera_joint: type fixed, parent arm1_camera_mount, child arm1_camera, origin xyz=0.03517 0 0 rpy=0.0 0 0
- added joint arm1_camera_mount: type fixed, parent arm1_mount_adapter, child arm1_camera_mount, origin xyz=-0.03485 0 0.09575 rpy=0 0 0
- added joint arm1_gripper1: type fixed, parent arm1_finger1_mount, child arm1_finger1, origin xyz=0 0 0 rpy=0 0 0
- added joint arm1_gripper1_mount: type prismatic, parent arm1_zimmer_body, child arm1_finger1_mount, origin xyz=0.00075 0.053 -0.011 rpy=3.1415 0 0, axis 0 1 0, limit lower=-0.007 upper=0.052 effort=150 velocity=0.01
- added joint arm1_gripper2: type fixed, parent arm1_finger2_mount, child arm1_finger2, origin xyz=0 0 0 rpy=0 0 0
- added joint arm1_gripper2_mount: type prismatic, parent arm1_zimmer_body, child arm1_finger2_mount, origin xyz=0.00075 -0.053 0.011 rpy=0 0 0, axis 0 1 0, limit lower=-0.007 upper=0.052 effort=150 velocity=0.01
- added joint arm1_gripper_adapter_joint: type fixed, parent arm1_mount_adapter, child arm1_gripper_adapter, origin xyz=0.0 0 0 rpy=0 0 0
- added joint arm1_j1: type revolute, parent arm1_link1, child arm1_link2, origin xyz=0 0 0.23605804505849792 rpy=0 0 1.0813043361136004e-07, axis 0 0 1, limit lower=-6.283185307179586 upper=6.283185307179586 effort=738.0 velocity=2.0943951023931953
- added joint arm1_j2: type revolute, parent arm1_link2, child arm1_link3, origin xyz=9.754030555240492e-05 0 0 rpy=1.5708629459765144 0 -4.880508667138009e-06, axis 0 0 1, limit lower=-6.283185307179586 upper=6.283185307179586 effort=738.0 velocity=2.0943951023931953
- added joint arm1_j3: type revolute, parent arm1_link3, child arm1_link4, origin xyz=-0.8610921552590647 0 0 rpy=0.0005884295412275638 -0.0004267141440094013 -7.335107699104623e-08, axis 0 0 1, limit lower=-3.141592653589793 upper=3.141592653589793 effort=433.0 velocity=2.6179938779914944
- added joint arm1_j4: type revolute, parent arm1_link4, child arm1_link5, origin xyz=-0.7278670242516039 0.00021723008103170053 0.19969583976195102 rpy=3.1405048492789644 3.141195896656006 -3.1415923332207147, axis 0 0 1, limit lower=-6.283185307179586 upper=6.283185307179586 effort=107.0 velocity=3.6651914291880923
- added joint arm1_j5: type revolute, parent arm1_link5, child arm1_link6, origin xyz=-3.309974135769099e-05 -0.159114862392224 -9.084549335387157e-05 rpy=1.57136726958501 0 7.582584195860861e-08, axis 0 0 1, limit lower=-6.283185307179586 upper=6.283185307179586 effort=107.0 velocity=3.6651914291880923
- added joint arm1_j6: type revolute, parent arm1_link6, child arm1_link7, origin xyz=-7.181658624943694e-05 0.1539659637667372 -4.189940789732904e-06 rpy=1.5707691133726167 3.141592653589793 3.1415924379608358, axis 0 0 1, limit lower=-6.283185307179586 upper=6.283185307179586 effort=107.0 velocity=3.6651914291880923
- added joint arm1_slide_tombstone_joint: type fixed, parent arm1_base_link, child arm1_slide_tombstone, origin xyz=0 0.095 0.1352 rpy=1.5708 0 3.14159
- added joint arm1_zimmer_body: type fixed, parent arm1_gripper_adapter, child arm1_zimmer_body, origin xyz=0.045 0 0 rpy=0 0 0
- added joint arm2_adapter_joint: type fixed, parent arm2_link7, child arm2_mount_adapter, origin xyz=0 -0.00317 0 rpy=1.5707963 -1.5707963 0
- added joint arm2_base_joint: type fixed, parent arm2_slide_tombstone, child arm2_link1, origin xyz=0 0 0 rpy=0 0 0
- added joint arm2_cable_harness_arm_link: type fixed, parent arm2_link3, child arm2_cable_harness_arm_link, origin xyz=0 0 0 rpy=0 0 0
- added joint arm2_cable_harness_ee_link: type fixed, parent arm2_link7, child arm2_cable_harness_ee_link, origin xyz=0 0 0 rpy=0 0 0
- added joint arm2_cable_harness_elbow_link: type fixed, parent arm2_link4, child arm2_cable_harness_elbow_link, origin xyz=0 0 0 rpy=0 0 0
- added joint arm2_camera_joint: type fixed, parent arm2_camera_mount, child arm2_camera, origin xyz=0.03517 0 0 rpy=0.0 0 0
- added joint arm2_camera_mount: type fixed, parent arm2_mount_adapter, child arm2_camera_mount, origin xyz=-0.03485 0 0.09575 rpy=0 0 0
- added joint arm2_gripper1: type fixed, parent arm2_finger1_mount, child arm2_finger1, origin xyz=0 0 0 rpy=0 0 0
- added joint arm2_gripper1_mount: type prismatic, parent arm2_zimmer_body, child arm2_finger1_mount, origin xyz=0.00075 0.053 -0.011 rpy=3.1415 0 0, axis 0 1 0, limit lower=-0.007 upper=0.052 effort=150 velocity=0.01
- added joint arm2_gripper2: type fixed, parent arm2_finger2_mount, child arm2_finger2, origin xyz=0 0 0 rpy=0 0 0
- added joint arm2_gripper2_mount: type prismatic, parent arm2_zimmer_body, child arm2_finger2_mount, origin xyz=0.00075 -0.053 0.011 rpy=0 0 0, axis 0 1 0, limit lower=-0.007 upper=0.052 effort=150 velocity=0.01
- added joint arm2_gripper_adapter_joint: type fixed, parent arm2_mount_adapter, child arm2_gripper_adapter, origin xyz=0.0 0 0 rpy=0 0 0
- added joint arm2_j1: type revolute, parent arm2_link1, child arm2_link2, origin xyz=0 0 0.23605804505849792 rpy=0 0 1.0813043361136004e-07, axis 0 0 1, limit lower=-6.283185307179586 upper=6.283185307179586 effort=738.0 velocity=2.0943951023931953
- added joint arm2_j2: type revolute, parent arm2_link2, child arm2_link3, origin xyz=9.754030555240492e-05 0 0 rpy=1.5708629459765144 0 -4.880508667138009e-06, axis 0 0 1, limit lower=-6.283185307179586 upper=6.283185307179586 effort=738.0 velocity=2.0943951023931953
- added joint arm2_j3: type revolute, parent arm2_link3, child arm2_link4, origin xyz=-0.8610921552590647 0 0 rpy=0.0005884295412275638 -0.0004267141440094013 -7.335107699104623e-08, axis 0 0 1, limit lower=-3.141592653589793 upper=3.141592653589793 effort=433.0 velocity=2.6179938779914944
- added joint arm2_j4: type revolute, parent arm2_link4, child arm2_link5, origin xyz=-0.7278670242516039 0.00021723008103170053 0.19969583976195102 rpy=3.1405048492789644 3.141195896656006 -3.1415923332207147, axis 0 0 1, limit lower=-6.283185307179586 upper=6.283185307179586 effort=107.0 velocity=3.6651914291880923
- added joint arm2_j5: type revolute, parent arm2_link5, child arm2_link6, origin xyz=-3.309974135769099e-05 -0.159114862392224 -9.084549335387157e-05 rpy=1.57136726958501 0 7.582584195860861e-08, axis 0 0 1, limit lower=-6.283185307179586 upper=6.283185307179586 effort=107.0 velocity=3.6651914291880923
- added joint arm2_j6: type revolute, parent arm2_link6, child arm2_link7, origin xyz=-7.181658624943694e-05 0.1539659637667372 -4.189940789732904e-06 rpy=1.5707691133726167 3.141592653589793 3.1415924379608358, axis 0 0 1, limit lower=-6.283185307179586 upper=6.283185307179586 effort=107.0 velocity=3.6651914291880923
- added joint arm2_slide_tombstone_joint: type fixed, parent arm2_base_link, child arm2_slide_tombstone, origin xyz=0 0.095 0.1352 rpy=1.5708 0 3.14159
- added joint arm2_zimmer_body: type fixed, parent arm2_gripper_adapter, child arm2_zimmer_body, origin xyz=0.045 0 0 rpy=0 0 0
- added joint arm3_adapter_joint: type fixed, parent arm3_link7, child arm3_mount_adapter, origin xyz=0 -0.00317 0 rpy=1.5707963 -1.5707963 0
- added joint arm3_base_joint: type fixed, parent arm3_slide_tombstone, child arm3_link1, origin xyz=0 0 0 rpy=0 0 0
- added joint arm3_cable_harness_arm_link: type fixed, parent arm3_link3, child arm3_cable_harness_arm_link, origin xyz=0 0 0 rpy=0 0 0
- added joint arm3_cable_harness_ee_link: type fixed, parent arm3_link7, child arm3_cable_harness_ee_link, origin xyz=0 0 0 rpy=0 0 0
- added joint arm3_cable_harness_elbow_link: type fixed, parent arm3_link4, child arm3_cable_harness_elbow_link, origin xyz=0 0 0 rpy=0 0 0
- added joint arm3_camera_joint: type fixed, parent arm3_camera_mount, child arm3_camera, origin xyz=0.03517 0 0 rpy=0.0 0 0
- added joint arm3_camera_mount: type fixed, parent arm3_mount_adapter, child arm3_camera_mount, origin xyz=-0.03485 0 0.09575 rpy=0 0 0
- added joint arm3_gripper1: type fixed, parent arm3_finger1_mount, child arm3_finger1, origin xyz=0 0 0 rpy=0 0 0
- added joint arm3_gripper1_mount: type prismatic, parent arm3_zimmer_body, child arm3_finger1_mount, origin xyz=0.00075 0.053 -0.011 rpy=3.1415 0 0, axis 0 1 0, limit lower=-0.007 upper=0.052 effort=150 velocity=0.01
- added joint arm3_gripper2: type fixed, parent arm3_finger2_mount, child arm3_finger2, origin xyz=0 0 0 rpy=0 0 0
- added joint arm3_gripper2_mount: type prismatic, parent arm3_zimmer_body, child arm3_finger2_mount, origin xyz=0.00075 -0.053 0.011 rpy=0 0 0, axis 0 1 0, limit lower=-0.007 upper=0.052 effort=150 velocity=0.01
- added joint arm3_gripper_adapter_joint: type fixed, parent arm3_mount_adapter, child arm3_gripper_adapter, origin xyz=0.0 0 0 rpy=0 0 0
- added joint arm3_j1: type revolute, parent arm3_link1, child arm3_link2, origin xyz=0 0 0.23605804505849792 rpy=0 0 1.0813043361136004e-07, axis 0 0 1, limit lower=-6.283185307179586 upper=6.283185307179586 effort=738.0 velocity=2.0943951023931953
- added joint arm3_j2: type revolute, parent arm3_link2, child arm3_link3, origin xyz=9.754030555240492e-05 0 0 rpy=1.5708629459765144 0 -4.880508667138009e-06, axis 0 0 1, limit lower=-6.283185307179586 upper=6.283185307179586 effort=738.0 velocity=2.0943951023931953
- added joint arm3_j3: type revolute, parent arm3_link3, child arm3_link4, origin xyz=-0.8610921552590647 0 0 rpy=0.0005884295412275638 -0.0004267141440094013 -7.335107699104623e-08, axis 0 0 1, limit lower=-3.141592653589793 upper=3.141592653589793 effort=433.0 velocity=2.6179938779914944
- added joint arm3_j4: type revolute, parent arm3_link4, child arm3_link5, origin xyz=-0.7278670242516039 0.00021723008103170053 0.19969583976195102 rpy=3.1405048492789644 3.141195896656006 -3.1415923332207147, axis 0 0 1, limit lower=-6.283185307179586 upper=6.283185307179586 effort=107.0 velocity=3.6651914291880923
- added joint arm3_j5: type revolute, parent arm3_link5, child arm3_link6, origin xyz=-3.309974135769099e-05 -0.159114862392224 -9.084549335387157e-05 rpy=1.57136726958501 0 7.582584195860861e-08, axis 0 0 1, limit lower=-6.283185307179586 upper=6.283185307179586 effort=107.0 velocity=3.6651914291880923
- added joint arm3_j6: type revolute, parent arm3_link6, child arm3_link7, origin xyz=-7.181658624943694e-05 0.1539659637667372 -4.189940789732904e-06 rpy=1.5707691133726167 3.141592653589793 3.1415924379608358, axis 0 0 1, limit lower=-6.283185307179586 upper=6.283185307179586 effort=107.0 velocity=3.6651914291880923
- added joint arm3_slide_tombstone_joint: type fixed, parent arm3_base_link, child arm3_slide_tombstone, origin xyz=0 0.095 0.1352 rpy=1.5708 0 3.14159
- added joint arm3_zimmer_body: type fixed, parent arm3_gripper_adapter, child arm3_zimmer_body, origin xyz=0.045 0 0 rpy=0 0 0
- added joint arm4_adapter_joint: type fixed, parent arm4_link7, child arm4_mount_adapter, origin xyz=0 -0.00317 0 rpy=1.5707963 -1.5707963 0
- added joint arm4_base_joint: type fixed, parent arm4_slide_tombstone, child arm4_link1, origin xyz=0 0 0 rpy=0 0 0
- added joint arm4_cable_harness_arm_link: type fixed, parent arm4_link3, child arm4_cable_harness_arm_link, origin xyz=0 0 0 rpy=0 0 0
- added joint arm4_cable_harness_ee_link: type fixed, parent arm4_link7, child arm4_cable_harness_ee_link, origin xyz=0 0 0 rpy=0 0 0
- added joint arm4_cable_harness_elbow_link: type fixed, parent arm4_link4, child arm4_cable_harness_elbow_link, origin xyz=0 0 0 rpy=0 0 0
- added joint arm4_camera_joint: type fixed, parent arm4_camera_mount, child arm4_camera, origin xyz=0.03517 0 0 rpy=0.0 0 0
- added joint arm4_camera_mount: type fixed, parent arm4_mount_adapter, child arm4_camera_mount, origin xyz=-0.03485 0 0.09575 rpy=0 0 0
- added joint arm4_gripper1: type fixed, parent arm4_finger1_mount, child arm4_finger1, origin xyz=0 0 0 rpy=0 0 0
- added joint arm4_gripper1_mount: type prismatic, parent arm4_zimmer_body, child arm4_finger1_mount, origin xyz=0.00075 0.053 -0.011 rpy=3.1415 0 0, axis 0 1 0, limit lower=-0.007 upper=0.052 effort=150 velocity=0.01
- added joint arm4_gripper2: type fixed, parent arm4_finger2_mount, child arm4_finger2, origin xyz=0 0 0 rpy=0 0 0
- added joint arm4_gripper2_mount: type prismatic, parent arm4_zimmer_body, child arm4_finger2_mount, origin xyz=0.00075 -0.053 0.011 rpy=0 0 0, axis 0 1 0, limit lower=-0.007 upper=0.052 effort=150 velocity=0.01
- added joint arm4_gripper_adapter_joint: type fixed, parent arm4_mount_adapter, child arm4_gripper_adapter, origin xyz=0.0 0 0 rpy=0 0 0
- added joint arm4_j1: type revolute, parent arm4_link1, child arm4_link2, origin xyz=0 0 0.23605804505849792 rpy=0 0 1.0813043361136004e-07, axis 0 0 1, limit lower=-6.283185307179586 upper=6.283185307179586 effort=738.0 velocity=2.0943951023931953
- added joint arm4_j2: type revolute, parent arm4_link2, child arm4_link3, origin xyz=9.754030555240492e-05 0 0 rpy=1.5708629459765144 0 -4.880508667138009e-06, axis 0 0 1, limit lower=-6.283185307179586 upper=6.283185307179586 effort=738.0 velocity=2.0943951023931953
- added joint arm4_j3: type revolute, parent arm4_link3, child arm4_link4, origin xyz=-0.8610921552590647 0 0 rpy=0.0005884295412275638 -0.0004267141440094013 -7.335107699104623e-08, axis 0 0 1, limit lower=-3.141592653589793 upper=3.141592653589793 effort=433.0 velocity=2.6179938779914944
- added joint arm4_j4: type revolute, parent arm4_link4, child arm4_link5, origin xyz=-0.7278670242516039 0.00021723008103170053 0.19969583976195102 rpy=3.1405048492789644 3.141195896656006 -3.1415923332207147, axis 0 0 1, limit lower=-6.283185307179586 upper=6.283185307179586 effort=107.0 velocity=3.6651914291880923
- added joint arm4_j5: type revolute, parent arm4_link5, child arm4_link6, origin xyz=-3.309974135769099e-05 -0.159114862392224 -9.084549335387157e-05 rpy=1.57136726958501 0 7.582584195860861e-08, axis 0 0 1, limit lower=-6.283185307179586 upper=6.283185307179586 effort=107.0 velocity=3.6651914291880923
- added joint arm4_j6: type revolute, parent arm4_link6, child arm4_link7, origin xyz=-7.181658624943694e-05 0.1539659637667372 -4.189940789732904e-06 rpy=1.5707691133726167 3.141592653589793 3.1415924379608358, axis 0 0 1, limit lower=-6.283185307179586 upper=6.283185307179586 effort=107.0 velocity=3.6651914291880923
- added joint arm4_slide_tombstone_joint: type fixed, parent arm4_base_link, child arm4_slide_tombstone, origin xyz=0 0.095 0.1352 rpy=1.5708 0 3.14159
- added joint arm4_zimmer_body: type fixed, parent arm4_gripper_adapter, child arm4_zimmer_body, origin xyz=0.045 0 0 rpy=0 0 0
- added joint plate_to_arm1: type fixed, parent slide_optical_plate, child arm1_base_link, origin xyz=0.357 0.357 0.0381 rpy=0 0 -0.78539816339
- added joint plate_to_arm2: type fixed, parent slide_optical_plate, child arm2_base_link, origin xyz=0.357 -0.357 0.0381 rpy=0 0 3.925
- added joint plate_to_arm3: type fixed, parent slide_optical_plate, child arm3_base_link, origin xyz=-0.357 0.357 0.0381 rpy=0 0 2.355
- added joint plate_to_arm4: type fixed, parent slide_optical_plate, child arm4_base_link, origin xyz=-0.4 -0.27 0.0646 rpy=0 0 3.1
- added joint slide_plate_joint: type fixed, parent slide_hexapod_plate, child slide_optical_plate, origin xyz=0 0 0.05715 rpy=0 0 0
