Commit message: Generate RSS platform usd

File: rss/rss_crab.urdf (robot description, URDF)
Before this commit: robot combined_hexapods, 86 links, 85 joints
Links:
- removed link slide_hexapod_plate
- added link base_link; collision mesh filename=meshes/mikrolar_description/slide_table.stl; visual mesh filename=meshes/mikrolar_description/slide_table.stl
- link slide_optical_plate: mass None -> 186.65
Joints:
- joint arm1_gripper1: axis (none) -> 0 1 0; child arm1_finger1 -> arm1_finger1_mount; limit (none) -> lower=-0.007 upper=0.052 effort=150 velocity=0.01; origin xyz=0 0 0 rpy=0 0 0 -> xyz=0.00075 0.053 -0.011 rpy=3.1415 0 0; parent arm1_finger1_mount -> arm1_zimmer_body; type fixed -> prismatic
- joint arm1_gripper1_mount: axis 0 1 0 -> (none); child arm1_finger1_mount -> arm1_finger1; limit lower=-0.007 upper=0.052 effort=150 velocity=0.01 -> (none); origin xyz=0.00075 0.053 -0.011 rpy=3.1415 0 0 -> xyz=0 0 0 rpy=0 0 0; parent arm1_zimmer_body -> arm1_finger1_mount; type prismatic -> fixed
- joint arm1_gripper2: axis (none) -> 0 1 0; child arm1_finger2 -> arm1_finger2_mount; limit (none) -> lower=-0.007 upper=0.052 effort=150 velocity=0.01; origin xyz=0 0 0 rpy=0 0 0 -> xyz=0.00075 -0.053 0.011 rpy=0 0 0; parent arm1_finger2_mount -> arm1_zimmer_body; type fixed -> prismatic
- joint arm1_gripper2_mount: axis 0 1 0 -> (none); child arm1_finger2_mount -> arm1_finger2; limit lower=-0.007 upper=0.052 effort=150 velocity=0.01 -> (none); origin xyz=0.00075 -0.053 0.011 rpy=0 0 0 -> xyz=0 0 0 rpy=0 0 0; parent arm1_zimmer_body -> arm1_finger2_mount; type prismatic -> fixed
- joint arm1_j1: limit lower=-6.283185307179586 upper=6.283185307179586 effort=738.0 velocity=2.0943951023931953 -> lower=-6.283185307179586 upper=6.283185307179586 effort=738.0 velocity=100
- joint arm1_j2: limit lower=-6.283185307179586 upper=6.283185307179586 effort=738.0 velocity=2.0943951023931953 -> lower=-6.283185307179586 upper=6.283185307179586 effort=738.0 velocity=100
- joint arm1_j3: limit lower=-3.141592653589793 upper=3.141592653589793 effort=433.0 velocity=2.6179938779914944 -> lower=-3.141592653589793 upper=3.141592653589793 effort=433.0 velocity=100
- joint arm1_j4: limit lower=-6.283185307179586 upper=6.283185307179586 effort=107.0 velocity=3.6651914291880923 -> lower=-6.283185307179586 upper=6.283185307179586 effort=107.0 velocity=100
- joint arm1_j5: limit lower=-6.283185307179586 upper=6.283185307179586 effort=107.0 velocity=3.6651914291880923 -> lower=-6.283185307179586 upper=6.283185307179586 effort=107.0 velocity=100
- joint arm1_j6: limit lower=-6.283185307179586 upper=6.283185307179586 effort=107.0 velocity=3.6651914291880923 -> lower=-6.283185307179586 upper=6.283185307179586 effort=107.0 velocity=100
- joint arm2_gripper1: axis (none) -> 0 1 0; child arm2_finger1 -> arm2_finger1_mount; limit (none) -> lower=-0.007 upper=0.052 effort=150 velocity=0.01; origin xyz=0 0 0 rpy=0 0 0 -> xyz=0.00075 0.053 -0.011 rpy=3.1415 0 0; parent arm2_finger1_mount -> arm2_zimmer_body; type fixed -> prismatic
- joint arm2_gripper1_mount: axis 0 1 0 -> (none); child arm2_finger1_mount -> arm2_finger1; limit lower=-0.007 upper=0.052 effort=150 velocity=0.01 -> (none); origin xyz=0.00075 0.053 -0.011 rpy=3.1415 0 0 -> xyz=0 0 0 rpy=0 0 0; parent arm2_zimmer_body -> arm2_finger1_mount; type prismatic -> fixed
- joint arm2_gripper2: axis (none) -> 0 1 0; child arm2_finger2 -> arm2_finger2_mount; limit (none) -> lower=-0.007 upper=0.052 effort=150 velocity=0.01; origin xyz=0 0 0 rpy=0 0 0 -> xyz=0.00075 -0.053 0.011 rpy=0 0 0; parent arm2_finger2_mount -> arm2_zimmer_body; type fixed -> prismatic
- joint arm2_gripper2_mount: axis 0 1 0 -> (none); child arm2_finger2_mount -> arm2_finger2; limit lower=-0.007 upper=0.052 effort=150 velocity=0.01 -> (none); origin xyz=0.00075 -0.053 0.011 rpy=0 0 0 -> xyz=0 0 0 rpy=0 0 0; parent arm2_zimmer_body -> arm2_finger2_mount; type prismatic -> fixed
- joint arm2_j1: limit lower=-6.283185307179586 upper=6.283185307179586 effort=738.0 velocity=2.0943951023931953 -> lower=-6.283185307179586 upper=6.283185307179586 effort=738.0 velocity=100
- joint arm2_j2: limit lower=-6.283185307179586 upper=6.283185307179586 effort=738.0 velocity=2.0943951023931953 -> lower=-6.283185307179586 upper=6.283185307179586 effort=738.0 velocity=100
- joint arm2_j3: limit lower=-3.141592653589793 upper=3.141592653589793 effort=433.0 velocity=2.6179938779914944 -> lower=-3.141592653589793 upper=3.141592653589793 effort=433.0 velocity=100
- joint arm2_j4: limit lower=-6.283185307179586 upper=6.283185307179586 effort=107.0 velocity=3.6651914291880923 -> lower=-6.283185307179586 upper=6.283185307179586 effort=107.0 velocity=100
- joint arm2_j5: limit lower=-6.283185307179586 upper=6.283185307179586 effort=107.0 velocity=3.6651914291880923 -> lower=-6.283185307179586 upper=6.283185307179586 effort=107.0 velocity=100
- joint arm2_j6: limit lower=-6.283185307179586 upper=6.283185307179586 effort=107.0 velocity=3.6651914291880923 -> lower=-6.283185307179586 upper=6.283185307179586 effort=107.0 velocity=100
- joint arm3_gripper1: axis (none) -> 0 1 0; child arm3_finger1 -> arm3_finger1_mount; limit (none) -> lower=-0.007 upper=0.052 effort=150 velocity=0.01; origin xyz=0 0 0 rpy=0 0 0 -> xyz=0.00075 0.053 -0.011 rpy=3.1415 0 0; parent arm3_finger1_mount -> arm3_zimmer_body; type fixed -> prismatic
- joint arm3_gripper1_mount: axis 0 1 0 -> (none); child arm3_finger1_mount -> arm3_finger1; limit lower=-0.007 upper=0.052 effort=150 velocity=0.01 -> (none); origin xyz=0.00075 0.053 -0.011 rpy=3.1415 0 0 -> xyz=0 0 0 rpy=0 0 0; parent arm3_zimmer_body -> arm3_finger1_mount; type prismatic -> fixed
- joint arm3_gripper2: axis (none) -> 0 1 0; child arm3_finger2 -> arm3_finger2_mount; limit (none) -> lower=-0.007 upper=0.052 effort=150 velocity=0.01; origin xyz=0 0 0 rpy=0 0 0 -> xyz=0.00075 -0.053 0.011 rpy=0 0 0; parent arm3_finger2_mount -> arm3_zimmer_body; type fixed -> prismatic
- joint arm3_gripper2_mount: axis 0 1 0 -> (none); child arm3_finger2_mount -> arm3_finger2; limit lower=-0.007 upper=0.052 effort=150 velocity=0.01 -> (none); origin xyz=0.00075 -0.053 0.011 rpy=0 0 0 -> xyz=0 0 0 rpy=0 0 0; parent arm3_zimmer_body -> arm3_finger2_mount; type prismatic -> fixed
- joint arm3_j1: limit lower=-6.283185307179586 upper=6.283185307179586 effort=738.0 velocity=2.0943951023931953 -> lower=-6.283185307179586 upper=6.283185307179586 effort=738.0 velocity=100
- joint arm3_j2: limit lower=-6.283185307179586 upper=6.283185307179586 effort=738.0 velocity=2.0943951023931953 -> lower=-6.283185307179586 upper=6.283185307179586 effort=738.0 velocity=100
- joint arm3_j3: limit lower=-3.141592653589793 upper=3.141592653589793 effort=433.0 velocity=2.6179938779914944 -> lower=-3.141592653589793 upper=3.141592653589793 effort=433.0 velocity=100
- joint arm3_j4: limit lower=-6.283185307179586 upper=6.283185307179586 effort=107.0 velocity=3.6651914291880923 -> lower=-6.283185307179586 upper=6.283185307179586 effort=107.0 velocity=100
- joint arm3_j5: limit lower=-6.283185307179586 upper=6.283185307179586 effort=107.0 velocity=3.6651914291880923 -> lower=-6.283185307179586 upper=6.283185307179586 effort=107.0 velocity=100
- joint arm3_j6: limit lower=-6.283185307179586 upper=6.283185307179586 effort=107.0 velocity=3.6651914291880923 -> lower=-6.283185307179586 upper=6.283185307179586 effort=107.0 velocity=100
- joint arm4_gripper1: axis (none) -> 0 1 0; child arm4_finger1 -> arm4_finger1_mount; limit (none) -> lower=-0.007 upper=0.052 effort=150 velocity=0.01; origin xyz=0 0 0 rpy=0 0 0 -> xyz=0.00075 0.053 -0.011 rpy=3.1415 0 0; parent arm4_finger1_mount -> arm4_zimmer_body; type fixed -> prismatic
- joint arm4_gripper1_mount: axis 0 1 0 -> (none); child arm4_finger1_mount -> arm4_finger1; limit lower=-0.007 upper=0.052 effort=150 velocity=0.01 -> (none); origin xyz=0.00075 0.053 -0.011 rpy=3.1415 0 0 -> xyz=0 0 0 rpy=0 0 0; parent arm4_zimmer_body -> arm4_finger1_mount; type prismatic -> fixed
- joint arm4_gripper2: axis (none) -> 0 1 0; child arm4_finger2 -> arm4_finger2_mount; limit (none) -> lower=-0.007 upper=0.052 effort=150 velocity=0.01; origin xyz=0 0 0 rpy=0 0 0 -> xyz=0.00075 -0.053 0.011 rpy=0 0 0; parent arm4_finger2_mount -> arm4_zimmer_body; type fixed -> prismatic
- joint arm4_gripper2_mount: axis 0 1 0 -> (none); child arm4_finger2_mount -> arm4_finger2; limit lower=-0.007 upper=0.052 effort=150 velocity=0.01 -> (none); origin xyz=0.00075 -0.053 0.011 rpy=0 0 0 -> xyz=0 0 0 rpy=0 0 0; parent arm4_zimmer_body -> arm4_finger2_mount; type prismatic -> fixed
- joint arm4_j1: limit lower=-6.283185307179586 upper=6.283185307179586 effort=738.0 velocity=2.0943951023931953 -> lower=-6.283185307179586 upper=6.283185307179586 effort=738.0 velocity=100
- joint arm4_j2: limit lower=-6.283185307179586 upper=6.283185307179586 effort=738.0 velocity=2.0943951023931953 -> lower=-6.283185307179586 upper=6.283185307179586 effort=738.0 velocity=100
- joint arm4_j3: limit lower=-3.141592653589793 upper=3.141592653589793 effort=433.0 velocity=2.6179938779914944 -> lower=-3.141592653589793 upper=3.141592653589793 effort=433.0 velocity=100
- joint arm4_j4: limit lower=-6.283185307179586 upper=6.283185307179586 effort=107.0 velocity=3.6651914291880923 -> lower=-6.283185307179586 upper=6.283185307179586 effort=107.0 velocity=100
- joint arm4_j5: limit lower=-6.283185307179586 upper=6.283185307179586 effort=107.0 velocity=3.6651914291880923 -> lower=-6.283185307179586 upper=6.283185307179586 effort=107.0 velocity=100
- joint arm4_j6: limit lower=-6.283185307179586 upper=6.283185307179586 effort=107.0 velocity=3.6651914291880923 -> lower=-6.283185307179586 upper=6.283185307179586 effort=107.0 velocity=100
- joint plate_to_arm1: origin xyz=0.357 0.357 0.0381 rpy=0 0 -0.78539816339 -> xyz=0.357 0.357 0.0381 rpy=0 0 -0.785
- joint plate_to_arm2: origin xyz=0.357 -0.357 0.0381 rpy=0 0 3.925 -> xyz=0.357 -0.357 0.0381 rpy=0 0 -2.358
- joint plate_to_arm3: origin xyz=-0.357 0.357 0.0381 rpy=0 0 2.355 -> xyz=-0.357 -0.357 0.0381 rpy=0 0 2.352
- joint plate_to_arm4: origin xyz=-0.4 -0.27 0.0646 rpy=0 0 3.1 -> xyz=-0.357 0.357 0.0381 rpy=0 0 0.781
- joint slide_plate_joint: parent slide_hexapod_plate -> base_link
