Commit message: added ur20 meshes, chaser and target imported into usd

File: rss/sim_chaser.urdf (robot description, URDF)
Before this commit: robot chaser_satellite, 74 links, 73 joints
Links:
- link chewie_alpha_base: geometry collision box size=0.018 0.015 0.027; collision cylinder length=0.032 radius=0.0065
- link chewie_base_link_inertia: geometry collision mesh filename=ur20_meshes/collision/base.stl; visual mesh filename=ur20_meshes/visual/base.dae
- link chewie_bravo_base: geometry collision box size=0.018 0.015 0.027; collision cylinder length=0.032 radius=0.0065
- link chewie_charlie_base: geometry collision box size=0.018 0.015 0.027; collision cylinder length=0.032 radius=0.0065
- link chewie_finger_mount_left: geometry collision mesh filename=rss_meshes/ZIMMER_SLIDE.STL; visual mesh filename=rss_meshes/ZIMMER_SLIDE.STL
- link chewie_finger_mount_right: geometry collision mesh filename=rss_meshes/ZIMMER_SLIDE.STL; visual mesh filename=rss_meshes/ZIMMER_SLIDE.STL
- link chewie_forearm_link: geometry collision mesh filename=ur20_meshes/collision/forearm.stl; visual mesh filename=ur20_meshes/visual/forearm.dae
- link chewie_gripper_adapter: geometry collision mesh filename=rss_meshes/GRIPPER_PLATE.STL; visual mesh filename=rss_meshes/GRIPPER_PLATE_VISUAL.STL
- link chewie_left_finger: geometry collision mesh filename=rss_meshes/Hex_Gripper.STL; visual mesh filename=rss_meshes/Hex_Gripper.STL
- link chewie_mount_adapter: geometry collision mesh filename=rss_meshes/MOUNT_PLATE.STL; visual mesh filename=rss_meshes/MOUNT_PLATE_VISUAL.STL
- link chewie_right_finger: geometry collision mesh filename=rss_meshes/Hex_Gripper.STL; visual mesh filename=rss_meshes/Hex_Gripper.STL
- link chewie_shoulder_link: geometry collision mesh filename=ur20_meshes/collision/shoulder.stl; visual mesh filename=ur20_meshes/visual/shoulder.dae
- link chewie_tombstone_base: geometry collision mesh filename=rss_meshes/tombstone.stl; visual mesh filename=rss_meshes/tombstone.stl
- link chewie_upper_arm_link: geometry collision mesh filename=ur20_meshes/collision/upperarm.stl; visual mesh filename=ur20_meshes/visual/upperarm.dae
- link chewie_wrist_1_link: geometry collision mesh filename=ur20_meshes/collision/wrist1.stl; visual mesh filename=ur20_meshes/visual/wrist1.dae
- link chewie_wrist_2_link: geometry collision mesh filename=ur20_meshes/collision/wrist2.stl; visual mesh filename=ur20_meshes/visual/wrist2.dae
- link chewie_wrist_3_link: geometry collision mesh filename=ur20_meshes/collision/wrist3.stl; visual mesh filename=ur20_meshes/visual/wrist3.dae
- link chewie_zimmer_body: geometry collision mesh filename=rss_meshes/ZIMMER_BOX.STL; visual mesh filename=rss_meshes/ZIMMER_BOX.STL
- link han_base_link_inertia: geometry collision mesh filename=ur20_meshes/collision/base.stl; visual mesh filename=ur20_meshes/visual/base.dae
- link han_camera: geometry collision mesh filename=rss_meshes/CAMERA.STL; visual mesh filename=rss_meshes/CAMERA_VISUAL_BASE.STL
- link han_camera_mount: geometry collision mesh filename=rss_meshes/CAMERA_MOUNT.STL; visual mesh filename=rss_meshes/CAMERA_MOUNT_VISUAL.STL
- link han_finger_mount_left: geometry collision mesh filename=rss_meshes/ZIMMER_SLIDE.STL; visual mesh filename=rss_meshes/ZIMMER_SLIDE.STL
- link han_finger_mount_right: geometry collision mesh filename=rss_meshes/ZIMMER_SLIDE.STL; visual mesh filename=rss_meshes/ZIMMER_SLIDE.STL
- link han_forearm_link: geometry collision mesh filename=ur20_meshes/collision/forearm.stl; visual mesh filename=ur20_meshes/visual/forearm.dae
- link han_gripper_adapter: geometry collision mesh filename=rss_meshes/GRIPPER_PLATE.STL; visual mesh filename=rss_meshes/GRIPPER_PLATE_VISUAL.STL
- link han_left_finger: geometry collision mesh filename=rss_meshes/Hex_Gripper.STL; visual mesh filename=rss_meshes/Hex_Gripper.STL
- link han_mount_adapter: geometry collision mesh filename=rss_meshes/MOUNT_PLATE.STL; visual mesh filename=rss_meshes/MOUNT_PLATE_VISUAL.STL
- link han_right_finger: geometry collision mesh filename=rss_meshes/Hex_Gripper.STL; visual mesh filename=rss_meshes/Hex_Gripper.STL
- link han_shoulder_link: geometry collision mesh filename=ur20_meshes/collision/shoulder.stl; visual mesh filename=ur20_meshes/visual/shoulder.dae
- link han_tombstone_base: geometry collision mesh filename=rss_meshes/tombstone.stl; visual mesh filename=rss_meshes/tombstone.stl
- link han_upper_arm_link: geometry collision mesh filename=ur20_meshes/collision/upperarm.stl; visual mesh filename=ur20_meshes/visual/upperarm.dae
- link han_wrist_1_link: geometry collision mesh filename=ur20_meshes/collision/wrist1.stl; visual mesh filename=ur20_meshes/visual/wrist1.dae
- link han_wrist_2_link: geometry collision mesh filename=ur20_meshes/collision/wrist2.stl; visual mesh filename=ur20_meshes/visual/wrist2.dae
- link han_wrist_3_link: geometry collision mesh filename=ur20_meshes/collision/wrist3.stl; visual mesh filename=ur20_meshes/visual/wrist3.dae
- link han_zimmer_body: geometry collision mesh filename=rss_meshes/ZIMMER_BOX.STL; visual mesh filename=rss_meshes/ZIMMER_BOX.STL
- link slide_coordinate_frame: geometry collision cylinder length=0.14 radius=0.01; collision cylinder length=0.14 radius=0.01

File: rss/sim_target.urdf (robot description, URDF)
Before this commit: robot target_satellite, 26 links, 25 joints
Links:
- link handle_1_mount: geometry visual mesh filename=rss_meshes/Hex_Grip_Collision.stl
- link handle_2_mount: geometry visual mesh filename=rss_meshes/Hex_Grip_Collision.stl
- link handle_3_mount: geometry visual mesh filename=rss_meshes/Hex_Grip_Collision.stl
- link handle_4_mount: geometry visual mesh filename=rss_meshes/Hex_Grip_Collision.stl
- link handle_5_mount: geometry visual mesh filename=rss_meshes/Hex_Grip_Collision.stl
- link rotary_FTS_Plate: geometry collision mesh filename=rss_meshes/FT_Plate_collision.stl; visual mesh filename=rss_meshes/FT_Plate.stl
- link rotary_coordinate_frame: geometry collision cylinder length=0.14 radius=0.01; collision cylinder length=0.14 radius=0.01
- link satellite_mockup: geometry collision mesh filename=rss_meshes/simple_satellite.stl; visual mesh filename=rss_meshes/simple_satellite.stl

Commit message: updated colors so they show up in usd

File: rss/sim_chaser.urdf (robot description, URDF)
Before this commit: robot chaser_satellite, 74 links, 73 joints
Joints:
- joint slide_optical_plate_joint: type floating -> fixed

File: rss/sim_target.urdf (robot description, URDF)
Before this commit: robot target_satellite, 26 links, 25 joints
Links:
- removed link base_link
Joints:
- removed joint rotary_optical_plate_joint
