Commit message: committing latest sim_chaser usd

File: rss/sim_chaser.urdf (robot description, URDF)
Before this commit: robot chaser_satellite, 74 links, 73 joints
Joints:
- joint ArmedFloating_Joint: origin xyz=0 0 0.705 rpy=0 0 0 -> xyz=0 0 0.705 rpy=0 0 0.7071

Commit message: updated sim_chaser.urdf with even simpler collision model

File: rss/sim_chaser.urdf (robot description, URDF)
Before this commit: robot chaser_satellite, 74 links, 73 joints
Links:
- link armed_mockup: geometry collision box size=1.0 1.0 1.0; visual box size=1.0 1.0 1.0
- link chewie_alpha_base: geometry visual mesh filename=rss_meshes/mounting.STL
- link chewie_base_link_inertia: geometry visual mesh filename=ur20_meshes/visual/base.dae
- link chewie_bota_lax_triplet_mount: geometry visual cylinder length=0.0254 radius=0.2159
- link chewie_bota_lax_triplet_top_plate: geometry visual cylinder length=0.0254 radius=0.2159
- link chewie_bravo_base: geometry visual mesh filename=rss_meshes/mounting.STL
- link chewie_cable_harness_arm_link: geometry visual box size=0.07 0.1524 0.07
- link chewie_cable_harness_ee_link: geometry visual box size=0.1778 0.0762 0.0254
- link chewie_cable_harness_elbow_link: geometry visual box size=0.15 0.0762 0.15
- link chewie_charlie_base: geometry visual mesh filename=rss_meshes/mounting.STL
- link chewie_finger_mount_left: geometry visual mesh filename=rss_meshes/ZIMMER_SLIDE.STL
- link chewie_finger_mount_right: geometry visual mesh filename=rss_meshes/ZIMMER_SLIDE.STL
- link chewie_forearm_link: geometry collision cylinder length=0.76 radius=0.05; visual mesh filename=ur20_meshes/visual/forearm.dae
- link chewie_gripper_adapter: geometry visual mesh filename=rss_meshes/GRIPPER_PLATE_VISUAL.STL
- link chewie_left_finger: geometry collision box size=0.085 0.0635 0.036351; visual mesh filename=rss_meshes/Hex_Gripper.STL
- link chewie_mount_adapter: geometry visual mesh filename=rss_meshes/MOUNT_PLATE_VISUAL.STL
- link chewie_right_finger: geometry collision box size=0.085 0.0635 0.036351; visual mesh filename=rss_meshes/Hex_Gripper.STL
- link chewie_shoulder_link: geometry collision cylinder length=0.2 radius=0.08; visual mesh filename=ur20_meshes/visual/shoulder.dae
- link chewie_tombstone_base: geometry visual mesh filename=rss_meshes/tombstone.stl
- link chewie_upper_arm_link: geometry collision cylinder length=0.861 radius=0.07; visual mesh filename=ur20_meshes/visual/upperarm.dae
- link chewie_wrist_1_link: geometry collision cylinder length=0.12 radius=0.045; visual mesh filename=ur20_meshes/visual/wrist1.dae
- link chewie_wrist_2_link: geometry collision cylinder length=0.12 radius=0.045; visual mesh filename=ur20_meshes/visual/wrist2.dae
- link chewie_wrist_3_link: geometry collision cylinder length=0.07 radius=0.045; visual mesh filename=ur20_meshes/visual/wrist3.dae
- link chewie_zimmer_body: geometry collision box size=0.045 0.13 0.062; visual mesh filename=rss_meshes/ZIMMER_BOX.STL
- link han_ati_omega191_mount: geometry visual box size=0.254 0.254 0.0254
- link han_ati_to_tombstone: geometry visual cylinder length=0.0254 radius=0.095
- link han_base_link_inertia: geometry visual mesh filename=ur20_meshes/visual/base.dae
- link han_cable_harness_arm_link: geometry visual box size=0.07 0.1524 0.07; visual cylinder length=0.8 radius=0.0381
- link han_cable_harness_ee_link: geometry visual box size=0.1778 0.0762 0.0254
- link han_cable_harness_elbow_link: geometry visual box size=0.15 0.0762 0.15
- link han_camera: geometry visual mesh filename=rss_meshes/CAMERA_VISUAL_BASE.STL; visual mesh filename=rss_meshes/CAMERA_VISUAL_FRAME.STL
- link han_camera_mount: geometry visual mesh filename=rss_meshes/CAMERA_MOUNT_VISUAL.STL
- link han_finger_mount_left: geometry visual mesh filename=rss_meshes/ZIMMER_SLIDE.STL
- link han_finger_mount_right: geometry visual mesh filename=rss_meshes/ZIMMER_SLIDE.STL
- link han_forearm_link: geometry collision cylinder length=0.76 radius=0.05; visual mesh filename=ur20_meshes/visual/forearm.dae
- link han_fts: geometry visual cylinder length=0.064 radius=0.095
- link han_gripper_adapter: geometry visual mesh filename=rss_meshes/GRIPPER_PLATE_VISUAL.STL
- link han_left_finger: geometry collision box size=0.085 0.0635 0.036351; visual mesh filename=rss_meshes/Hex_Gripper.STL
- link han_mount_adapter: geometry visual mesh filename=rss_meshes/MOUNT_PLATE_VISUAL.STL
- link han_right_finger: geometry collision box size=0.085 0.0635 0.036351; visual mesh filename=rss_meshes/Hex_Gripper.STL
- link han_shoulder_link: geometry collision cylinder length=0.2 radius=0.08; visual mesh filename=ur20_meshes/visual/shoulder.dae
- link han_tombstone_base: geometry visual mesh filename=rss_meshes/tombstone.stl
- link han_upper_arm_link: geometry collision cylinder length=0.861 radius=0.07; visual mesh filename=ur20_meshes/visual/upperarm.dae
- link han_wrist_1_link: geometry collision cylinder length=0.12 radius=0.045; visual mesh filename=ur20_meshes/visual/wrist1.dae
- link han_wrist_2_link: geometry collision cylinder length=0.12 radius=0.045; visual mesh filename=ur20_meshes/visual/wrist2.dae
- link han_wrist_3_link: geometry collision cylinder length=0.07 radius=0.045; visual mesh filename=ur20_meshes/visual/wrist3.dae
- link han_zimmer_body: geometry collision box size=0.045 0.13 0.062; visual mesh filename=rss_meshes/ZIMMER_BOX.STL
- link slide_coordinate_frame: geometry visual cylinder length=0.14 radius=0.01; visual cylinder length=0.14 radius=0.01

File: rss/sim_chewie.urdf (robot description, URDF)
Before this commit: robot chewie_arm, 42 links, 41 joints
Links:
- link chewie_alpha_base: geometry visual mesh filename=rss_meshes/mounting.STL
- link chewie_base_link_inertia: geometry collision cylinder length=0.109 radius=0.1225; visual mesh filename=ur20_meshes/visual/base.dae
- link chewie_bota_lax_triplet_mount: geometry visual cylinder length=0.0254 radius=0.2159
- link chewie_bota_lax_triplet_top_plate: geometry visual cylinder length=0.0254 radius=0.2159
- link chewie_bravo_base: geometry visual mesh filename=rss_meshes/mounting.STL
- link chewie_cable_harness_arm_link: geometry visual box size=0.07 0.1524 0.07
- link chewie_cable_harness_ee_link: geometry visual box size=0.1778 0.0762 0.0254
- link chewie_cable_harness_elbow_link: geometry visual box size=0.15 0.0762 0.15
- link chewie_charlie_base: geometry visual mesh filename=rss_meshes/mounting.STL
- link chewie_finger_mount_left: geometry visual mesh filename=rss_meshes/ZIMMER_SLIDE.STL
- link chewie_finger_mount_right: geometry visual mesh filename=rss_meshes/ZIMMER_SLIDE.STL
- link chewie_forearm_link: geometry collision cylinder length=0.728 radius=0.075; visual mesh filename=ur20_meshes/visual/forearm.dae
- link chewie_gripper_adapter: geometry visual mesh filename=rss_meshes/GRIPPER_PLATE_VISUAL.STL
- link chewie_left_finger: geometry collision box size=0.092905 0.0635 0.036351; visual mesh filename=rss_meshes/Hex_Gripper.STL
- link chewie_mount_adapter: geometry visual mesh filename=rss_meshes/MOUNT_PLATE_VISUAL.STL
- link chewie_right_finger: geometry collision box size=0.092905 0.0635 0.036351; visual mesh filename=rss_meshes/Hex_Gripper.STL
- link chewie_shoulder_link: geometry collision cylinder length=0.224 radius=0.095; visual mesh filename=ur20_meshes/visual/shoulder.dae
- link chewie_tombstone_base: geometry collision box size=0.18977 0.245 0.2577; visual mesh filename=rss_meshes/tombstone.stl
- link chewie_upper_arm_link: geometry collision cylinder length=0.861 radius=0.09; visual mesh filename=ur20_meshes/visual/upperarm.dae
- link chewie_wrist_1_link: geometry collision cylinder length=0.137 radius=0.055; visual mesh filename=ur20_meshes/visual/wrist1.dae
- link chewie_wrist_2_link: geometry collision cylinder length=0.138 radius=0.055; visual mesh filename=ur20_meshes/visual/wrist2.dae
- link chewie_wrist_3_link: geometry collision cylinder length=0.07 radius=0.053; visual mesh filename=ur20_meshes/visual/wrist3.dae
- link chewie_zimmer_body: geometry collision box size=0.045 0.13 0.062; visual mesh filename=rss_meshes/ZIMMER_BOX.STL
- link slide_coordinate_frame: geometry visual cylinder length=0.14 radius=0.01; visual cylinder length=0.14 radius=0.01
