Commit message: restored effort and velocity limits from 300 and 100 to 10 and 10, added back front and back sensor links

File: crab/crab.urdf (robot description, URDF)
Before this commit: robot CRAB_Model_Assembly, 33 links, 32 joints
Links:
- added link back_sensor_link, mass 1e-10; visual box size=0.01 0.06 0.04
- added link front_sensor_link, mass 1e-10; visual box size=0.01 0.06 0.04
Joints:
- added joint back_sensor_link_joint: type fixed, parent base_link, child back_sensor_link, origin xyz=-0.28 0 -0.01 rpy=0 0 0
- added joint front_sensor_link_joint: type fixed, parent base_link, child front_sensor_link, origin xyz=0.28 0 -0.01 rpy=0 0 0
- joint arm1_j1: limit lower=-3.14 upper=3.14 effort=300 velocity=100 -> lower=-3.14 upper=3.14 effort=10 velocity=10
- joint arm1_j2: limit lower=-0.174 upper=3.14 effort=300 velocity=100 -> lower=-0.174 upper=3.14 effort=10 velocity=10
- joint arm1_j3: limit lower=-3.14 upper=3.14 effort=300 velocity=100 -> lower=-3.14 upper=3.14 effort=10 velocity=10
- joint arm1_j4: limit lower=-3.14 upper=0.174 effort=300 velocity=100 -> lower=-3.14 upper=0.174 effort=10 velocity=10
- joint arm1_j5: limit lower=-3.14 upper=3.14 effort=300 velocity=100 -> lower=-3.14 upper=3.14 effort=10 velocity=10
- joint arm1_j6: limit lower=-0.174 upper=3.14 effort=300 velocity=100 -> lower=-0.174 upper=3.14 effort=10 velocity=10
- joint arm1_j7: limit lower=-3.14 upper=3.14 effort=300 velocity=100 -> lower=-3.14 upper=3.14 effort=10 velocity=10
- joint arm2_j1: limit lower=-3.14 upper=3.14 effort=300 velocity=100 -> lower=-3.14 upper=3.14 effort=10 velocity=10
- joint arm2_j2: limit lower=-0.174 upper=3.14 effort=300 velocity=100 -> lower=-0.174 upper=3.14 effort=10 velocity=10
- joint arm2_j3: limit lower=-3.14 upper=3.14 effort=300 velocity=100 -> lower=-3.14 upper=3.14 effort=10 velocity=10
- joint arm2_j4: limit lower=-3.14 upper=0.174 effort=300 velocity=100 -> lower=-3.14 upper=0.174 effort=10 velocity=10
- joint arm2_j5: limit lower=-3.14 upper=3.14 effort=300 velocity=100 -> lower=-3.14 upper=3.14 effort=10 velocity=10
- joint arm2_j6: limit lower=-0.174 upper=3.14 effort=300 velocity=100 -> lower=-0.174 upper=3.14 effort=10 velocity=10
- joint arm2_j7: limit lower=-3.14 upper=3.14 effort=300 velocity=100 -> lower=-3.14 upper=3.14 effort=10 velocity=10
- joint arm3_j1: limit lower=-3.14 upper=3.14 effort=300 velocity=100 -> lower=-3.14 upper=3.14 effort=10 velocity=10
- joint arm3_j2: limit lower=-0.174 upper=3.14 effort=300 velocity=100 -> lower=-0.174 upper=3.14 effort=10 velocity=10
- joint arm3_j3: limit lower=-3.14 upper=3.14 effort=300 velocity=100 -> lower=-3.14 upper=3.14 effort=10 velocity=10
- joint arm3_j4: limit lower=-3.14 upper=0.174 effort=300 velocity=100 -> lower=-3.14 upper=0.174 effort=10 velocity=10
- joint arm3_j5: limit lower=-3.14 upper=3.14 effort=300 velocity=100 -> lower=-3.14 upper=3.14 effort=10 velocity=10
- joint arm3_j6: limit lower=-0.174 upper=3.14 effort=300 velocity=100 -> lower=-0.174 upper=3.14 effort=10 velocity=10
- joint arm3_j7: limit lower=-3.14 upper=3.14 effort=300 velocity=100 -> lower=-3.14 upper=3.14 effort=10 velocity=10
- joint arm4_j1: limit lower=-3.14 upper=3.14 effort=300 velocity=100 -> lower=-3.14 upper=3.14 effort=10 velocity=10
- joint arm4_j2: limit lower=-0.174 upper=3.14 effort=300 velocity=100 -> lower=-0.174 upper=3.14 effort=10 velocity=10
- joint arm4_j3: limit lower=-3.14 upper=3.14 effort=300 velocity=100 -> lower=-3.14 upper=3.14 effort=10 velocity=10
- joint arm4_j4: limit lower=-3.14 upper=0.174 effort=300 velocity=100 -> lower=-3.14 upper=0.174 effort=10 velocity=10
- joint arm4_j5: limit lower=-3.14 upper=3.14 effort=300 velocity=100 -> lower=-3.14 upper=3.14 effort=10 velocity=10
- joint arm4_j6: limit lower=-0.174 upper=3.14 effort=300 velocity=100 -> lower=-0.174 upper=3.14 effort=10 velocity=10
- joint arm4_j7: limit lower=-3.14 upper=3.14 effort=300 velocity=100 -> lower=-3.14 upper=3.14 effort=10 velocity=10

Commit message: updated collision geometry to old model with crab feet

File: crab/crab.urdf (robot description, URDF)
Before this commit: robot CRAB_Model_Assembly, 35 links, 34 joints
Links:
- link arm1_link2: geometry collision cylinder length=0.05 radius=0.04; visual mesh filename=meshes/arm1_link2.STL
- link arm1_link3: geometry collision cylinder length=0.05 radius=0.03; visual mesh filename=meshes/arm1_link3.STL
- link arm1_link4: geometry collision cylinder length=0.05 radius=0.03; visual mesh filename=meshes/arm1_link4.STL
- link arm1_link6: geometry collision cylinder length=0.05 radius=0.02; visual mesh filename=meshes/arm1_link6.STL
- link arm2_link2: geometry collision cylinder length=0.05 radius=0.04; visual mesh filename=meshes/arm2_link2.STL
- link arm2_link3: geometry collision cylinder length=0.05 radius=0.03; visual mesh filename=meshes/arm2_link3.STL
- link arm2_link4: geometry collision cylinder length=0.05 radius=0.03; visual mesh filename=meshes/arm2_link4.STL
- link arm2_link6: geometry collision cylinder length=0.05 radius=0.02; visual mesh filename=meshes/arm2_link6.STL
- link arm3_link2: geometry collision cylinder length=0.05 radius=0.04; visual mesh filename=meshes/arm3_link2.STL
- link arm3_link3: geometry collision cylinder length=0.05 radius=0.03; visual mesh filename=meshes/arm3_link3.STL
- link arm3_link4: geometry collision cylinder length=0.05 radius=0.03; visual mesh filename=meshes/arm3_link4.STL
- link arm3_link6: geometry collision cylinder length=0.05 radius=0.02; visual mesh filename=meshes/arm3_link6.STL
- link arm4_link2: geometry collision cylinder length=0.05 radius=0.04; visual mesh filename=meshes/arm4_link2.STL
- link arm4_link3: geometry collision cylinder length=0.05 radius=0.03; visual mesh filename=meshes/arm4_link3.STL
- link arm4_link4: geometry collision cylinder length=0.05 radius=0.03; visual mesh filename=meshes/arm4_link4.STL
- link arm4_link6: geometry collision cylinder length=0.05 radius=0.02; visual mesh filename=meshes/arm4_link6.STL
- link base_link: geometry collision box size=0.4 0.4 0.15; visual mesh filename=meshes/base_link.STL

Commit message: Fix roll joints on crab legs

File: crab/crab.urdf (robot description, URDF)
Before this commit: robot CRAB_Model_Assembly, 33 links, 32 joints
Joints:
- joint arm1_j3: limit lower=-3.14 upper=3.14 effort=300 velocity=100 -> lower=0 upper=0 effort=300 velocity=100
- joint arm1_j5: limit lower=-3.14 upper=3.14 effort=300 velocity=100 -> lower=0 upper=0 effort=300 velocity=100
- joint arm1_j7: limit lower=-3.14 upper=3.14 effort=300 velocity=100 -> lower=0 upper=0 effort=300 velocity=100
- joint arm2_j3: limit lower=-3.14 upper=3.14 effort=300 velocity=100 -> lower=0 upper=0 effort=300 velocity=100
- joint arm2_j5: limit lower=-3.14 upper=3.14 effort=300 velocity=100 -> lower=0 upper=0 effort=300 velocity=100
- joint arm2_j7: limit lower=-3.14 upper=3.14 effort=300 velocity=100 -> lower=0 upper=0 effort=300 velocity=100
- joint arm3_j3: limit lower=-3.14 upper=3.14 effort=300 velocity=100 -> lower=0 upper=0 effort=300 velocity=100
- joint arm3_j5: limit lower=-3.14 upper=3.14 effort=300 velocity=100 -> lower=0 upper=0 effort=300 velocity=100
- joint arm3_j7: limit lower=-3.14 upper=3.14 effort=300 velocity=100 -> lower=0 upper=0 effort=300 velocity=100
- joint arm4_j3: limit lower=-3.14 upper=3.14 effort=300 velocity=100 -> lower=0 upper=0 effort=300 velocity=100
- joint arm4_j5: limit lower=-3.14 upper=3.14 effort=300 velocity=100 -> lower=0 upper=0 effort=300 velocity=100
- joint arm4_j7: limit lower=-3.14 upper=3.14 effort=300 velocity=100 -> lower=0 upper=0 effort=300 velocity=100

Commit message: Fix j6 (ankle pitch)

File: crab/crab.urdf (robot description, URDF)
Before this commit: robot CRAB_Model_Assembly, 33 links, 32 joints
Joints:
- joint arm1_j6: limit lower=-0.174 upper=3.14 effort=300 velocity=100 -> lower=0 upper=0 effort=300 velocity=100; origin xyz=0.10239375 0.000793749999999789 0.0254 rpy=0 0 0 -> xyz=0.10239375 0.000793749999999789 0.0254 rpy=0 0.5 0
- joint arm2_j6: limit lower=-0.174 upper=3.14 effort=300 velocity=100 -> lower=0 upper=0 effort=300 velocity=100; origin xyz=0.10239375 -0.000793749999999754 -0.0254000000000001 rpy=0 0 0 -> xyz=0.10239375 -0.000793749999999754 -0.0254000000000001 rpy=0 0.5 0
- joint arm3_j6: limit lower=-0.174 upper=3.14 effort=300 velocity=100 -> lower=0 upper=0 effort=300 velocity=100; origin xyz=-0.10239375 0.000793749999999791 -0.0254 rpy=0 0 0 -> xyz=-0.10239375 0.000793749999999791 -0.0254 rpy=0 0.5 0
- joint arm4_j6: limit lower=-0.174 upper=3.14 effort=300 velocity=100 -> lower=0 upper=0 effort=300 velocity=100; origin xyz=-0.10239375 -0.000793749999999786 0.0254 rpy=0 0 0 -> xyz=-0.10239375 -0.000793749999999786 0.0254 rpy=0 0.5 0

Commit message: Adjust j6 joint angle

File: crab/crab.urdf (robot description, URDF)
Before this commit: robot CRAB_Model_Assembly, 33 links, 32 joints
Joints:
- joint arm1_j6: origin xyz=0.10239375 0.000793749999999789 0.0254 rpy=0 0.5 0 -> xyz=0.10239375 0.000793749999999789 0.0254 rpy=0 0 0
- joint arm2_j6: origin xyz=0.10239375 -0.000793749999999754 -0.0254000000000001 rpy=0 0.5 0 -> xyz=0.10239375 -0.000793749999999754 -0.0254000000000001 rpy=0 0 0
- joint arm3_j6: origin xyz=-0.10239375 0.000793749999999791 -0.0254 rpy=0 0.5 0 -> xyz=-0.10239375 0.000793749999999791 -0.0254 rpy=0 0 0
- joint arm4_j6: origin xyz=-0.10239375 -0.000793749999999786 0.0254 rpy=0 0.5 0 -> xyz=-0.10239375 -0.000793749999999786 0.0254 rpy=0 0 0

Commit message: Reenable ankle links

File: crab/crab.urdf (robot description, URDF)
Before this commit: robot CRAB_Model_Assembly, 33 links, 32 joints
Joints:
- joint arm1_j3: limit lower=0 upper=0 effort=300 velocity=100 -> lower=-3.14 upper=3.14 effort=300 velocity=100
- joint arm1_j5: limit lower=0 upper=0 effort=300 velocity=100 -> lower=-3.14 upper=3.14 effort=300 velocity=100
- joint arm1_j6: limit lower=0 upper=0 effort=300 velocity=100 -> lower=-0.174 upper=3.14 effort=300 velocity=100
- joint arm1_j7: limit lower=0 upper=0 effort=300 velocity=100 -> lower=-3.14 upper=3.14 effort=300 velocity=100
- joint arm2_j3: limit lower=0 upper=0 effort=300 velocity=100 -> lower=-3.14 upper=3.14 effort=300 velocity=100
- joint arm2_j5: limit lower=0 upper=0 effort=300 velocity=100 -> lower=-3.14 upper=3.14 effort=300 velocity=100
- joint arm2_j6: limit lower=0 upper=0 effort=300 velocity=100 -> lower=-0.174 upper=3.14 effort=300 velocity=100
- joint arm2_j7: limit lower=0 upper=0 effort=300 velocity=100 -> lower=-3.14 upper=3.14 effort=300 velocity=100
- joint arm3_j3: limit lower=0 upper=0 effort=300 velocity=100 -> lower=-3.14 upper=3.14 effort=300 velocity=100
- joint arm3_j5: limit lower=0 upper=0 effort=300 velocity=100 -> lower=-3.14 upper=3.14 effort=300 velocity=100
- joint arm3_j6: limit lower=0 upper=0 effort=300 velocity=100 -> lower=-0.174 upper=3.14 effort=300 velocity=100
- joint arm3_j7: limit lower=0 upper=0 effort=300 velocity=100 -> lower=-3.14 upper=3.14 effort=300 velocity=100
- joint arm4_j3: limit lower=0 upper=0 effort=300 velocity=100 -> lower=-3.14 upper=3.14 effort=300 velocity=100
- joint arm4_j5: limit lower=0 upper=0 effort=300 velocity=100 -> lower=-3.14 upper=3.14 effort=300 velocity=100
- joint arm4_j6: limit lower=0 upper=0 effort=300 velocity=100 -> lower=-0.174 upper=3.14 effort=300 velocity=100
- joint arm4_j7: limit lower=0 upper=0 effort=300 velocity=100 -> lower=-3.14 upper=3.14 effort=300 velocity=100

Commit message: Change j6 offset to 0.2

File: crab/crab.urdf (robot description, URDF)
Before this commit: robot CRAB_Model_Assembly, 33 links, 32 joints
Joints:
- joint arm1_j3: limit lower=-3.14 upper=3.14 effort=300 velocity=100 -> lower=0 upper=0 effort=300 velocity=100
- joint arm1_j5: limit lower=-3.14 upper=3.14 effort=300 velocity=100 -> lower=0 upper=0 effort=300 velocity=100
- joint arm1_j6: limit lower=-0.174 upper=3.14 effort=300 velocity=100 -> lower=0 upper=0 effort=300 velocity=100; origin xyz=0.10239375 0.000793749999999789 0.0254 rpy=0 0 0 -> xyz=0.10239375 0.000793749999999789 0.0254 rpy=0 0.2 0
- joint arm1_j7: limit lower=-3.14 upper=3.14 effort=300 velocity=100 -> lower=0 upper=0 effort=300 velocity=100
- joint arm2_j3: limit lower=-3.14 upper=3.14 effort=300 velocity=100 -> lower=0 upper=0 effort=300 velocity=100
- joint arm2_j5: limit lower=-3.14 upper=3.14 effort=300 velocity=100 -> lower=0 upper=0 effort=300 velocity=100
- joint arm2_j6: limit lower=-0.174 upper=3.14 effort=300 velocity=100 -> lower=0 upper=0 effort=300 velocity=100; origin xyz=0.10239375 -0.000793749999999754 -0.0254000000000001 rpy=0 0 0 -> xyz=0.10239375 -0.000793749999999754 -0.0254000000000001 rpy=0 0.2 0
- joint arm2_j7: limit lower=-3.14 upper=3.14 effort=300 velocity=100 -> lower=0 upper=0 effort=300 velocity=100
- joint arm3_j3: limit lower=-3.14 upper=3.14 effort=300 velocity=100 -> lower=0 upper=0 effort=300 velocity=100
- joint arm3_j5: limit lower=-3.14 upper=3.14 effort=300 velocity=100 -> lower=0 upper=0 effort=300 velocity=100
- joint arm3_j6: limit lower=-0.174 upper=3.14 effort=300 velocity=100 -> lower=0 upper=0 effort=300 velocity=100; origin xyz=-0.10239375 0.000793749999999791 -0.0254 rpy=0 0 0 -> xyz=-0.10239375 0.000793749999999791 -0.0254 rpy=0 0.2 0
- joint arm3_j7: limit lower=-3.14 upper=3.14 effort=300 velocity=100 -> lower=0 upper=0 effort=300 velocity=100
- joint arm4_j3: limit lower=-3.14 upper=3.14 effort=300 velocity=100 -> lower=0 upper=0 effort=300 velocity=100
- joint arm4_j5: limit lower=-3.14 upper=3.14 effort=300 velocity=100 -> lower=0 upper=0 effort=300 velocity=100
- joint arm4_j6: limit lower=-0.174 upper=3.14 effort=300 velocity=100 -> lower=0 upper=0 effort=300 velocity=100; origin xyz=-0.10239375 -0.000793749999999786 0.0254 rpy=0 0 0 -> xyz=-0.10239375 -0.000793749999999786 0.0254 rpy=0 0.2 0
- joint arm4_j7: limit lower=-3.14 upper=3.14 effort=300 velocity=100 -> lower=0 upper=0 effort=300 velocity=100

Commit message: Increase joint limits on hip pitch

File: crab/crab.urdf (robot description, URDF)
Before this commit: robot CRAB_Model_Assembly, 33 links, 32 joints
Joints:
- joint arm1_j2: limit lower=-0.174 upper=3.14 effort=300 velocity=100 -> lower=-1.57 upper=3.14 effort=300 velocity=100
- joint arm2_j2: limit lower=-0.174 upper=3.14 effort=300 velocity=100 -> lower=-1.57 upper=3.14 effort=300 velocity=100
- joint arm3_j2: limit lower=-0.174 upper=3.14 effort=300 velocity=100 -> lower=-1.57 upper=3.14 effort=300 velocity=100
- joint arm4_j2: limit lower=-0.174 upper=3.14 effort=300 velocity=100 -> lower=-1.57 upper=3.14 effort=300 velocity=100

Commit message: Replace hip roll with hip yaw

File: crab/crab.urdf (robot description, URDF)
Before this commit: robot CRAB_Model_Assembly, 33 links, 32 joints
Links:
- link arm1_link4: geometry visual mesh filename=meshes/arm1_link4.STL
- link arm2_link4: geometry visual mesh filename=meshes/arm2_link4.STL
- link arm3_link4: geometry visual mesh filename=meshes/arm3_link4.STL
- link arm4_link4: geometry visual mesh filename=meshes/arm4_link4.STL
Joints:
- joint arm1_j1: axis 1 0 0 -> 0 0 1; limit lower=-3.14 upper=3.14 effort=300 velocity=100 -> lower=-0.785 upper=1.57 effort=300 velocity=100; origin xyz=0.127 -0.1778 0 rpy=1.5707963267949 0 0 -> xyz=0.127 -0.1778 0 rpy=3.14 0 0
- joint arm2_j1: axis 1 0 0 -> 0 0 1; limit lower=-3.14 upper=3.14 effort=300 velocity=100 -> lower=-0.785 upper=1.57 effort=300 velocity=100; origin xyz=0.127 0.1778 0 rpy=1.5708 0 0 -> xyz=0.127 0.1778 0 rpy=0 0 0
- joint arm3_j1: axis -1 0 0 -> 0 0 1; limit lower=-3.14 upper=3.14 effort=300 velocity=100 -> lower=-1.57 upper=0.785 effort=300 velocity=100; origin xyz=-0.127 0.1778 0 rpy=1.5708 0 0 -> xyz=-0.127 0.1778 0 rpy=0 0 0
- joint arm4_j1: axis -1 0 0 -> 0 0 1; limit lower=-3.14 upper=3.14 effort=300 velocity=100 -> lower=-1.57 upper=0.785 effort=300 velocity=100; origin xyz=-0.127 -0.1778 0 rpy=1.5707963267949 0 0 -> xyz=-0.127 -0.1778 0 rpy=3.14 0 0

Commit message: Update collision meshes in crab urdf (self collisions must be disabled)

File: crab/crab.urdf (robot description, URDF)
Before this commit: robot CRAB_Model_Assembly, 33 links, 32 joints
Links:
- link arm1_link2: geometry collision cylinder length=0.112 radius=0.038; visual mesh filename=meshes/arm1_link2.STL
- link arm1_link3: geometry collision cylinder length=0.15 radius=0.031; visual mesh filename=meshes/arm1_link3.STL
- link arm1_link4: geometry collision cylinder length=0.09 radius=0.0325; visual mesh filename=meshes/arm1_link4.STL
- link arm1_link5: geometry collision cylinder length=0.15 radius=0.025; visual mesh filename=meshes/arm1_link5.STL
- link arm1_link6: geometry collision cylinder length=0.067 radius=0.026; visual mesh filename=meshes/arm1_link6.STL
- link arm2_link2: geometry collision cylinder length=0.112 radius=0.038; visual mesh filename=meshes/arm2_link2.STL
- link arm2_link3: geometry collision cylinder length=0.15 radius=0.031; visual mesh filename=meshes/arm2_link3.STL
- link arm2_link4: geometry collision cylinder length=0.09 radius=0.0325; visual mesh filename=meshes/arm2_link4.STL
- link arm2_link5: geometry collision cylinder length=0.15 radius=0.025; visual mesh filename=meshes/arm2_link5.STL
- link arm2_link6: geometry collision cylinder length=0.067 radius=0.026; visual mesh filename=meshes/arm2_link6.STL
- link arm3_link2: geometry collision cylinder length=0.112 radius=0.038; visual mesh filename=meshes/arm3_link2.STL
- link arm3_link3: geometry collision cylinder length=0.15 radius=0.031; visual mesh filename=meshes/arm3_link3.STL
- link arm3_link4: geometry collision cylinder length=0.09 radius=0.0325; visual mesh filename=meshes/arm3_link4.STL
- link arm3_link5: geometry collision cylinder length=0.15 radius=0.025; visual mesh filename=meshes/arm3_link5.STL
- link arm3_link6: geometry collision cylinder length=0.067 radius=0.026; visual mesh filename=meshes/arm3_link6.STL
- link arm4_link2: geometry collision cylinder length=0.112 radius=0.038; visual mesh filename=meshes/arm4_link2.STL
- link arm4_link3: geometry collision cylinder length=0.15 radius=0.031; visual mesh filename=meshes/arm4_link3.STL
- link arm4_link4: geometry collision cylinder length=0.09 radius=0.0325; visual mesh filename=meshes/arm4_link4.STL
- link arm4_link5: geometry collision cylinder length=0.15 radius=0.025; visual mesh filename=meshes/arm4_link5.STL
- link arm4_link6: geometry collision cylinder length=0.067 radius=0.026; visual mesh filename=meshes/arm4_link6.STL
Joints:
- joint arm1_j6: origin xyz=0.10239375 0.000793749999999789 0.0254 rpy=0 0.2 0 -> xyz=0.10239375 0.000793749999999789 0.0254 rpy=0 0 0
- joint arm2_j6: origin xyz=0.10239375 -0.000793749999999754 -0.0254000000000001 rpy=0 0.2 0 -> xyz=0.10239375 -0.000793749999999754 -0.0254000000000001 rpy=0 0 0
- joint arm3_j6: origin xyz=-0.10239375 0.000793749999999791 -0.0254 rpy=0 0.2 0 -> xyz=-0.10239375 0.000793749999999791 -0.0254 rpy=0 0 0
- joint arm4_j6: origin xyz=-0.10239375 -0.000793749999999786 0.0254 rpy=0 0.2 0 -> xyz=-0.10239375 -0.000793749999999786 0.0254 rpy=0 0 0

Commit message: Adjust joint limits and collision meshes so self collisions are feasible

File: crab/crab.urdf (robot description, URDF)
Before this commit: robot CRAB_Model_Assembly, 33 links, 32 joints
Links:
- link arm1_link2: geometry collision cylinder length=0.03 radius=0.038; visual mesh filename=meshes/arm1_link2.STL
- link arm1_link3: geometry collision cylinder length=0.062 radius=0.0325; collision cylinder length=0.09 radius=0.031
- link arm1_link4: geometry visual mesh filename=meshes/arm1_link4.STL
- link arm1_link5: geometry collision cylinder length=0.067 radius=0.026; collision cylinder length=0.11 radius=0.025
- link arm1_link6: geometry visual mesh filename=meshes/arm1_link6.STL
- link arm2_link2: geometry collision cylinder length=0.03 radius=0.038; visual mesh filename=meshes/arm2_link2.STL
- link arm2_link3: geometry collision cylinder length=0.062 radius=0.0325; collision cylinder length=0.09 radius=0.031
- link arm2_link4: geometry visual mesh filename=meshes/arm2_link4.STL
- link arm2_link5: geometry collision cylinder length=0.067 radius=0.026; collision cylinder length=0.11 radius=0.025
- link arm2_link6: geometry visual mesh filename=meshes/arm2_link6.STL
- link arm3_link2: geometry collision cylinder length=0.03 radius=0.038; visual mesh filename=meshes/arm3_link2.STL
- link arm3_link3: geometry collision cylinder length=0.062 radius=0.0325; collision cylinder length=0.09 radius=0.031
- link arm3_link4: geometry visual mesh filename=meshes/arm3_link4.STL
- link arm3_link5: geometry collision cylinder length=0.067 radius=0.026; collision cylinder length=0.11 radius=0.025
- link arm3_link6: geometry visual mesh filename=meshes/arm3_link6.STL
- link arm4_link2: geometry collision cylinder length=0.03 radius=0.038; visual mesh filename=meshes/arm4_link2.STL
- link arm4_link3: geometry collision cylinder length=0.062 radius=0.0325; collision cylinder length=0.09 radius=0.031
- link arm4_link4: geometry visual mesh filename=meshes/arm4_link4.STL
- link arm4_link5: geometry collision cylinder length=0.067 radius=0.026; collision cylinder length=0.11 radius=0.025
- link arm4_link6: geometry visual mesh filename=meshes/arm4_link6.STL
Joints:
- joint arm1_j1: limit lower=-0.785 upper=1.57 effort=300 velocity=100 -> lower=-0.34 upper=0.785 effort=300 velocity=100
- joint arm1_j4: limit lower=-3.14 upper=0.174 effort=300 velocity=100 -> lower=-3.14 upper=0 effort=300 velocity=100
- joint arm1_j6: limit lower=-0.174 upper=3.14 effort=300 velocity=100 -> lower=-0.174 upper=3.05 effort=300 velocity=100
- joint arm2_j1: limit lower=-0.785 upper=1.57 effort=300 velocity=100 -> lower=-0.3 upper=0.785 effort=300 velocity=100
- joint arm2_j4: limit lower=-3.14 upper=0.174 effort=300 velocity=100 -> lower=-3.14 upper=0 effort=300 velocity=100
- joint arm2_j6: limit lower=-0.174 upper=3.14 effort=300 velocity=100 -> lower=-0.174 upper=3.05 effort=300 velocity=100
- joint arm3_j1: limit lower=-1.57 upper=0.785 effort=300 velocity=100 -> lower=-0.785 upper=0.34 effort=300 velocity=100
- joint arm3_j4: limit lower=-3.14 upper=0.174 effort=300 velocity=100 -> lower=-3.14 upper=0 effort=300 velocity=100
- joint arm3_j6: limit lower=-0.174 upper=3.14 effort=300 velocity=100 -> lower=-0.174 upper=3.05 effort=300 velocity=100
- joint arm4_j1: limit lower=-1.57 upper=0.785 effort=300 velocity=100 -> lower=-0.785 upper=0.3 effort=300 velocity=100
- joint arm4_j4: limit lower=-3.14 upper=0.174 effort=300 velocity=100 -> lower=-3.14 upper=0 effort=300 velocity=100
- joint arm4_j6: limit lower=-0.174 upper=3.14 effort=300 velocity=100 -> lower=-0.174 upper=3.05 effort=300 velocity=100
