Commit message: Increase hip yaw limits

File: crab/crab.urdf (robot description, URDF)
Before this commit: robot CRAB_Model_Assembly, 33 links, 32 joints
Links:
- link base_link: geometry collision box size=0.4 0.4 0.2; visual mesh filename=meshes/base_link.STL
Joints:
- joint arm1_j1: limit lower=-0.34 upper=0.785 effort=300 velocity=100 -> lower=-0.34 upper=1.57 effort=300 velocity=100
- joint arm2_j1: limit lower=-0.3 upper=0.785 effort=300 velocity=100 -> lower=-0.34 upper=1.57 effort=300 velocity=100
- joint arm3_j1: limit lower=-0.785 upper=0.34 effort=300 velocity=100 -> lower=-1.57 upper=0.34 effort=300 velocity=100
- joint arm4_j1: limit lower=-0.785 upper=0.3 effort=300 velocity=100 -> lower=-1.57 upper=0.34 effort=300 velocity=100

Commit message: Fix ankle pitch joint

File: crab/crab.urdf (robot description, URDF)
Before this commit: robot CRAB_Model_Assembly, 33 links, 32 joints
Joints:
- joint arm1_j6: axis 0 -1 0 -> (none); limit lower=-0.174 upper=3.05 effort=300 velocity=100 -> (none); type revolute -> fixed
- joint arm2_j6: axis 0 1 0 -> (none); limit lower=-0.174 upper=3.05 effort=300 velocity=100 -> (none); type revolute -> fixed
- joint arm3_j6: axis 0 -1 0 -> (none); limit lower=-0.174 upper=3.05 effort=300 velocity=100 -> (none); type revolute -> fixed
- joint arm4_j6: axis 0 1 0 -> (none); limit lower=-0.174 upper=3.05 effort=300 velocity=100 -> (none); type revolute -> fixed
